File: cad_files/mm5d/mm5d.sch (KiCad schematic (older format))
At the start: 1 part

Commit message: 190920
Parts:
- added P? (x24): SCREW_CONN_1, symbol SCREW_CONN_1
- added U4, U5: Relay_panel, symbol Relay_panel
Connections:
- new net: P?.1, U4.~ (VCCJb) (x12)
- new net: P?.1, U5.~ (VCCJb) (x12)
- new net OUT1: U5.~ (VCCJb)
- new net OUT2: U5.~ (VCCJb)
- new net OUT3: U5.~ (VCCJb)
- new net OUT4: U5.~ (VCCJb)
- new net OUT5: U4.~ (VCCJb)
- new net OUT6: U4.~ (VCCJb)
- new net OUT7: U4.~ (VCCJb)
- new net OUT8: U4.~ (VCCJb)
Other:
- moved on the sheet: J?

Commit message: 190920
Parts:
- removed P? (x23): SCREW_CONN_1, symbol SCREW_CONN_1
- added F1: 2,5A F, symbol Fuse
- added P1, P10, P11, P12, P13, P14, P15, P16, P17, P18, P19, P2, P20, P21, P22, P23, P24, P26, P27, P28, P29, P3, P30, P31, P32, P33, P34, P35, P36, P4, P5, P6, P7, P8, P9: SCREW_CONN_1, symbol SCREW_CONN_1
- gave numbers to parts that had none: 2
Connections:
- net Connecting unit/GND: now also P37.5
- net Connecting unit/RXD: now also P37.2
- net Connecting unit/TXD: now also P37.3
- net Input unit/+5V: now also P11.1
- net Input unit/GND: now also P12.1
- new net: P13.1, U4.~ (VCCJb)
- new net: P14.1, U4.~ (VCCJb)
- new net: P15.1, U4.~ (VCCJb)
- new net: P16.1, U4.~ (VCCJb)
- new net: P17.1, U4.~ (VCCJb)
- new net: P18.1, U4.~ (VCCJb)
- new net: P19.1, U4.~ (VCCJb)
- new net: P20.1, U4.~ (VCCJb)
- new net: P21.1, U4.~ (VCCJb)
- new net: P22.1, U4.~ (VCCJb)
- new net: P23.1, U4.~ (VCCJb)
- new net: P24.1, U4.~ (VCCJb)
- new net: P26.1, U5.~ (VCCJb)
- new net: P27.1, U5.~ (VCCJb)
- new net: P28.1, U5.~ (VCCJb)
- new net: P29.1, U5.~ (VCCJb)
- new net: P30.1, U5.~ (VCCJb)
- new net: P31.1, U5.~ (VCCJb)
- new net: P32.1, U5.~ (VCCJb)
- new net: P33.1, U5.~ (VCCJb)
- new net: P34.1, U5.~ (VCCJb)
- new net: P35.1, U5.~ (VCCJb)
- new net: P36.1, U5.~ (VCCJb)
- new net: F1.2, P1.1
- new net +5V-2: U5.~ (VCCJb)
- new net +5V-3: U4.~ (VCCJb)
- new net Connecting unit/+5V-IN: F1.1
- new net GND: P2.1, P3.1
- new net GND-2: U5.~ (VCCJb)
- new net GND-3: U4.~ (VCCJb)
- new net Input unit/GND: P4.1
- new net Input unit/IN1: P5.1
- new net Input unit/IN2: P6.1
- new net Input unit/IN3: P7.1
- new net Input unit/IN4: P8.1
- new net Input unit/S1: P9.1
- new net Input unit/S2: P10.1
- no-connect marks 0 -> 6
Other:
- note added: "5V DC\nPELV"
- note added: "Console\nRS-232"
- note added: "Inputs"
- note added: "Outputs"
- note added: "Power in"
- note added: "U2"
- note added: "U2 Connecting unit is connencted to Raspberry Pi with a 40 wire cable.\n This connection is not on this diagram."
- note added: "U3"
- note added: "U4"
- note added: "U5"
- note added: "U6"
- moved on the sheet: P25, P37

Commit message: 190922
Connections:
- net labels added: +3,3V-2, DS1, DS2
- net labels removed: DATA-S1, DATA-S2
- wire segments 154 -> 161
Other:
- note added: "5V DC"
- note removed: "5V DC\nPELV"
- moved on the sheet: F1, P10, P11, P12, P13, P14, P15, P16, P17, P18, P19, P20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

Commit message: 190922
Connections:
- wire segments 161 -> 159
Changed lines of the file:
@@
 F0 "Connecting unit" 60
 F1 "u2.sch" 60
-F2 "GPIO2" B L 2875 2325 60
-F3 "GPIO3" B L 2875 2425 60
-F4 "GPIO4" B L 2875 2525 60
-F5 "GPIO5" B L 2875 2625 60
-F6 "GPIO6" B L 2875 2725 60
-F7 "GPIO12" B L 2875 2825 60
-F8 "GPIO13" B L 2875 2925 60
-F9 "TXD" B R 4025 2725 60
-F10 "RXD" B R 4025 2825 60
-F11 "GPIO16" B L 2875 3025 60
+F2 "GPIO2" O L 2875 2325 60
+F3 "GPIO3" O L 2875 2425 60
+F4 "GPIO4" O L 2875 2525 60
+F5 "GPIO5" O L 2875 2625 60
+F6 "GPIO6" O L 2875 2725 60
+F7 "GPIO12" O L 2875 2825 60
+F8 "GPIO13" O L 2875 2925 60
+F9 "TXD" O R 4025 2725 60
+F10 "RXD" I R 4025 2825 60
+F11 "GPIO16" O L 2875 3025 60
 F12 "GPIO17" B L 2875 3125 60
 F13 "GPIO18" B L 2875 3225 60
-F14 "GPIO19" B L 2875 3325 60
-F15 "GPIO20" B L 2875 3425 60
-F16 "GPIO21" B L 2875 3525 60
-F17 "GPIO22" B L 2875 3625 60
-F18 "GPIO23" B L 2875 3725 60
-F19 "GPIO24" B L 2875 3825 60
-F20 "GPIO25" B L 2875 3925 60
+F14 "GPIO19" O L 2875 3325 60
+F15 "GPIO20" O L 2875 3425 60
+F16 "GPIO21" O L 2875 3525 60
+F17 "GPIO22" I L 2875 3625 60
+F18 "GPIO23" I L 2875 3725 60
+F19 "GPIO24" I L 2875 3825 60
+F20 "GPIO25" O L 2875 3925 60
 F21 "GPIO26" B L 2875 4025 60
-F22 "GPIO27" B L 2875 4125 60
+F22 "GPIO27" I L 2875 4125 60
 F23 "MOSI" B R 4025 2325 60
 F24 "CE0" O R 4025 2425 60
@@
 	4325 2325 4025 2325
 Wire Bus Line
-	2475 4975 2475 6775
-Wire Bus Line
-	2475 6775 2475 6875
-Wire Bus Line
-	2475 6875 2475 6975
-Wire Bus Line
-	2475 6975 2475 7575
-Wire Bus Line
-	2475 7575 2475 7675
-Wire Bus Line
-	2475 7675 2475 7775
-Wire Bus Line
-	2475 7775 2475 7875
-Wire Bus Line
-	2475 7875 2475 7975
-Wire Bus Line
-	2475 7975 2475 8075
-Wire Bus Line
-	2475 8075 2475 8175
-Wire Bus Line
-	2475 8175 2475 8275
-Wire Bus Line
-	2475 8275 2475 8375
+	2475 4975 2475 8375
 Wire Wire Line
 	1850 6875 2375 6875
@@
 	2375 7075 1850 7075
 Wire Bus Line
-	3075 7325 3075 7425
-Wire Bus Line
-	3075 7425 3075 7525
-Wire Bus Line
-	3075 7525 3075 7625
-Wire Bus Line
-	3075 7625 3075 8050
+	3075 7325 3075 8050
 Wire Bus Line
 	3075 8050 3975 8050
 Wire Bus Line
-	3975 8050 3975 8500
-Wire Bus Line
-	3975 8500 3975 8600
-Wire Bus Line
-	3975 8600 3975 8700
-Wire Bus Line
-	3975 8700 3975 8800
+	3975 8050 3975 8800
 Wire Wire Line
 	2875 2825 1725 2825
@@
 	1625 4975 2475 4975
 Wire Bus Line
-	1625 2050 1625 2725
-Wire Bus Line
-	1625 2725 1625 2825
-Wire Bus Line
-	1625 2825 1625 2925
-Wire Bus Line
-	1625 2925 1625 3025
-Wire Bus Line
-	1625 3025 1625 3125
-Wire Bus Line
-	1625 3125 1625 3425
-Wire Bus Line
-	1625 3425 1625 3525
-Wire Bus Line
-	1625 3525 1625 3625
-Wire Bus Line
-	1625 3625 1625 4025
-Wire Bus Line
-	1625 4025 1625 4975
+	1625 2050 1625 4975
 Wire Wire Line
 	1350 2325 2875 2325
@@
 	2875 2525 1350 2525
 Wire Bus Line
-	4650 7725 4650 7900
-Wire Bus Line
-	4650 7900 4650 8000
-Wire Bus Line
-	4650 8000 4650 8100
-Wire Bus Line
-	4650 8100 4650 8200
-Wire Bus Line
-	4650 8200 4650 8300
-Wire Bus Line
-	4650 8300 4650 8400
-Wire Bus Line
-	1250 2425 1250 2525
-Wire Bus Line
-	1250 2525 1250 2625
-Wire Bus Line
-	1250 2625 1250 4325
-Wire Bus Line
-	1250 4325 1250 5200
+	4650 7725 4650 8400
+Wire Bus Line
+	1250 2425 1250 5200
 Wire Bus Line
 	1250 5200 4100 5200
 Wire Bus Line
-	4100 5200 4100 6375
-Wire Bus Line
-	4100 6375 4100 6475
-Wire Bus Line
-	4100 6475 4100 6575
-Wire Bus Line
-	4100 6575 4100 6675
+	4100 5200 4100 6675
 Wire Bus Line
 	1625 2050 4425 2050
 Wire Bus Line
-	4425 2050 4425 2225
-Wire Bus Line
-	4425 2225 4425 2325
-Wire Bus Line
-	4425 2325 4425 2425
+	4425 2050 4425 2425
 Wire Wire Line
 	5400 4900 5275 4900
@@
 	5275 5100 5400 5100
 Wire Bus Line
-	5175 3025 5175 3125
-Wire Bus Line
-	5175 3125 5175 3225
-Wire Bus Line
-	5175 3225 5175 3325
-Wire Bus Line
-	5175 3325 5175 4700
-Wire Bus Line
-	5175 4700 5175 4800
-Wire Bus Line
-	5175 4800 5175 4900
-Wire Bus Line
-	5175 4900 5175 5000
+	5175 3025 5175 5000
 Wire Wire Line
 	5400 4800 5275 4800
@@
 	4200 6775 5400 6775
 Wire Bus Line
-	2250 4725 2350 4725
-Wire Bus Line
-	2350 4725 2450 4725
-Wire Bus Line
-	2450 4725 2550 4725
-Wire Bus Line
-	2550 4725 2650 4725
-Wire Bus Line
-	2650 4725 2750 4725
-Wire Bus Line
-	2750 4725 3975 4725
+	2250 4725 3975 4725
 Wire Bus Line
 	3975 4725 3975 7725
@@
 	7250 7550 5600 7550
 Wire Wire Line
-	6525 7800 6800 7800
-Wire Wire Line
-	6525 7900 6800 7900
-Wire Wire Line
-	6525 8000 6800 8000
-Wire Wire Line
-	6525 8100 6800 8100
-Wire Wire Line
-	6525 8200 6800 8200
-Wire Wire Line
-	6525 8300 6800 8300
-Wire Wire Line
-	6525 8400 6800 8400
-Wire Wire Line
-	6525 8500 6800 8500
-Wire Wire Line
-	6525 8600 6800 8600
+	6575 7800 6800 7800
+Wire Wire Line
+	6575 7900 6800 7900
+Wire Wire Line
+	6575 8000 6800 8000
+Wire Wire Line
+	6575 8100 6800 8100
+Wire Wire Line
+	6575 8200 6800 8200
+Wire Wire Line
+	6575 8300 6800 8300
+Wire Wire Line
+	6575 8400 6800 8400
+Wire Wire Line
+	6575 8500 6800 8500
+Wire Wire Line
+	6575 8600 6800 8600
 Wire Wire Line
 	4025 2725 5300 2725
@@
 	6425 3425 6800 3425
 Wire Wire Line
-	4750 3525 6650 3525
-Wire Wire Line
-	6650 3525 6800 3525
+	4750 3525 6800 3525
 Text HLabel 4025 4125 0    60   UnSpc ~ 0
 GND-1
@@
 	6800 3625 6650 3625
 Wire Wire Line
-	6650 3525 6650 3625
-Wire Wire Line
-	6650 3625 6650 3700
+	6650 3525 6650 3700
 Text Notes 6825 4150 0    60   ~ 0
 Outputs
