File: cad_files/mm5d/mm5d.sch (KiCad schematic (older format))
At the start: 40 parts, among them P1 SCREW_CONN_1, P10 SCREW_CONN_1, P11 SCREW_CONN_1, P12 SCREW_CONN_1, P13 SCREW_CONN_1, P14 SCREW_CONN_1, P15 SCREW_CONN_1, P16 SCREW_CONN_1, P17 SCREW_CONN_1, P18 SCREW_CONN_1, P19 SCREW_CONN_1, P2 SCREW_CONN_1, P20 SCREW_CONN_1, P21 SCREW_CONN_1, P22 SCREW_CONN_1, P23 SCREW_CONN_1, P24 SCREW_CONN_1, P25 SCREW_CONN_1, P26 SCREW_CONN_1, P27 SCREW_CONN_1, P28 SCREW_CONN_1, P29 SCREW_CONN_1, P3 SCREW_CONN_1, P30 SCREW_CONN_1, P31 SCREW_CONN_1, P32 SCREW_CONN_1, P33 SCREW_CONN_1, P34 SCREW_CONN_1, P35 SCREW_CONN_1, P36 SCREW_CONN_1, P37 DB9, P4 SCREW_CONN_1, P5 SCREW_CONN_1, P6 SCREW_CONN_1, P7 SCREW_CONN_1, P8 SCREW_CONN_1, P9 SCREW_CONN_1, U4 Relay_panel, U5 Relay_panel

Commit message: 190923
Changed lines of the file:
@@
 $EndSheet
 $Sheet
-S 950  6775 900  2150
+S 950  6775 900  2300
 U 5D5B105C
 F0 "Display unit" 60
 F1 "u6.sch" 60
-F2 "+5V" I R 1850 8625 60
-F3 "GND" U R 1850 8825 60
+F2 "+5V" I R 1850 8775 60
+F3 "GND" U R 1850 8975 60
 F4 "MOSI" I R 1850 6875 60
 F5 "CE0" I R 1850 6975 60
@@
 F18 "LED12" I R 1850 8375 60
 F19 "LED13" I R 1850 8475 60
-F20 "+3.3V" I R 1850 8725 60
+F20 "+3.3V" I R 1850 8875 60
+F21 "SW-MODE" I R 1850 8625 60
 $EndSheet
 $Comp
@@
 	4325 2325 4025 2325
 Wire Bus Line
-	2475 4975 2475 8375
+	2475 4975 2475 8525
 Wire Wire Line
 	1850 6875 2375 6875
@@
 +3,3V-1
 Wire Wire Line
-	1850 8625 3275 8625
-Wire Wire Line
-	3275 8625 3275 4825
+	1850 8775 3275 8775
+Wire Wire Line
+	3275 8775 3275 4825
 Wire Wire Line
 	3275 4825 4450 4825
@@
 	4450 3725 4025 3725
 Wire Wire Line
-	3375 8725 1850 8725
-Wire Wire Line
-	3375 4925 3375 8725
+	3375 8875 1850 8875
+Wire Wire Line
+	3375 4925 3375 8875
 Wire Wire Line
 	3375 4925 4350 4925
@@
 	4250 5025 3475 5025
 Wire Wire Line
-	3475 5025 3475 8825
-Wire Wire Line
-	3475 8825 1850 8825
+	3475 5025 3475 8975
+Wire Wire Line
+	3475 8975 1850 8975
 Wire Wire Line
 	4025 3825 5300 3825
@@
 Wire Wire Line
 	4550 9000 5700 9000
-Text Notes 950  9100 0    60   ~ 0
+Text Notes 950  9250 0    60   ~ 0
 U6
 Text Notes 2875 4675 0    60   ~ 0
@@
 Wire Wire Line
 	4850 3625 4025 3625
+Entry Wire Line
+	1625 4125 1725 4025
+Text Label 1725 4025 0    60   ~ 0
+SW-MODE
+Wire Wire Line
+	1725 4025 2875 4025
+Text Label 2375 8625 2    60   ~ 0
+SW-MODE
+Entry Wire Line
+	2375 8625 2475 8525
+Wire Wire Line
+	1850 8625 2375 8625
 $EndSCHEMATC

Commit message: 190925
Parts:
- added D1: 1N5408, symbol D
Connections:
- net Connecting unit/+5V-IN: now also D1.1 (K)
- net GND: now also D1.2 (A)
Changed lines of the file:
@@
 NoConn ~ 6550 2125
 Wire Wire Line
-	6800 3625 6650 3625
+	6450 3625 6800 3625
 Wire Wire Line
 	6650 3525 6650 3700
@@
 Wire Wire Line
 	1850 8625 2375 8625
+$Comp
+L D D1
+U 1 1 5D8B1D7E
+P 6300 3625
+F 0 "D1" H 6175 3550 50  0000 C CNN
+F 1 "1N5408" H 6300 3450 50  0000 C CNN
+F 2 "" H 6300 3625 50  0000 C CNN
+F 3 "" H 6300 3625 50  0000 C CNN
+	1    6300 3625
+	1    0    0    -1
+$EndComp
+Wire Wire Line
+	6150 3625 6050 3625
+Wire Wire Line
+	6050 3625 6050 3425
+Connection ~ 6050 3425
 $EndSCHEMATC
