File: cad_files/mm5d/mm5d.sch (KiCad schematic (older format))
At the start: 46 parts, among them P1 SCREW_CONN_1, P10 SCREW_CONN_1, P11 SCREW_CONN_1, P12 SCREW_CONN_1, P13 SCREW_CONN_1, P14 SCREW_CONN_1, P15 SCREW_CONN_1, P16 SCREW_CONN_1, P17 SCREW_CONN_1, P18 SCREW_CONN_1, P19 SCREW_CONN_1, P2 SCREW_CONN_1, P20 SCREW_CONN_1, P21 SCREW_CONN_1, P22 SCREW_CONN_1, P23 SCREW_CONN_1, P24 SCREW_CONN_1, P25 SCREW_CONN_1, P26 SCREW_CONN_1, P27 SCREW_CONN_1, P28 SCREW_CONN_1, P29 SCREW_CONN_1, P3 SCREW_CONN_1, P30 SCREW_CONN_1, P31 SCREW_CONN_1, P32 SCREW_CONN_1, P33 SCREW_CONN_1, P34 SCREW_CONN_1, P35 SCREW_CONN_1, P36 SCREW_CONN_1, P37 DB9, P4 CONN_02X20, P4 SCREW_CONN_1, P5 CONN_02X20, P5 SCREW_CONN_1, P6 CONN_02X20, P6 SCREW_CONN_1, P7 SCREW_CONN_1, P8 SCREW_CONN_1, P9 SCREW_CONN_1, U4 Relay_panel, U5 Relay_panel

Commit message: 200128
Parts:
- removed P10, P11, P12, P13, P14, P15, P16, P17, P18, P19, P20, P21, P22, P23, P24, P25, P26, P27, P28, P29, P30, P31, P32, P33, P34, P35, P36, P4, P5, P6, P7, P8, P9: SCREW_CONN_1, symbol SCREW_CONN_1
- removed U4, U?: Relay_panel, symbol Relay_panel
- added U6: Relay_panel, symbol Relay_panel
- gave numbers to parts that had none: 1
- renumbered U5 to U7
Connections:
- net labels added: GPIO02, GPIO03, GPIO04
- net labels removed: +3,3V-1, +3,3V-2, +5V-1, +5V-2, +5V-3, +5V-4, CEO, DS1, DS2, GND-1, GND-2, GND-3, GND-4, GND-IN, IN1, IN2, IN3, IN4, LED-ACT, LED-ERR1, LED-ERR2, LED-ERR3, LED-ERR4, LED-IN1, LED-IN2, LED-IN3, LED-IN4, LED-OUT1, LED-OUT2, LED-OUT3, LED-OUT4, OUT1, OUT2, OUT3, OUT4, OUT5, OUT6, OUT7, OUT8, SW-MODE, U2-U4, U2-U5, U2-U6, U3-U2, U3-U6
- wire segments 233 -> 139
- no-connect marks 25 -> 55
Other:
- note removed: "Inputs"
- note removed: "Outputs"
- note removed: "U2"
- note removed: "U3"
- note removed: "U5"
- note removed: "U6"
- moved on the sheet: D1, F1, P1, P2, P3, P37, P4, P5, P6, U3

Commit message: 200129
Parts:
- removed P1, P2, P3: SCREW_CONN_1, symbol SCREW_CONN_1
- added J1: Screw_Terminal_1x02, symbol Screw_Terminal_1x02
Connections:
- net labels added: GPIO18, RXD, TXD
- wire segments 139 -> 189
- no-connect marks 55 -> 75
Other:
- note added: "Console"
- note added: "Inputs"
- note added: "LEDs"
- note added: "Matrix display"
- note added: "Outputs"
- note removed: "5V DC"
- note removed: "Console\nRS-232"
- note removed: "U2 Connecting unit is connencted to Raspberry Pi with a 40 wire cable.\n This connection is not on this diagram."
- note removed: "U4"
- moved on the sheet: D1, F1, P37, P4, P5, P6, U3, U6, U7

Commit message: 200130
Parts:
- removed J1: Screw_Terminal_1x02, symbol Screw_Terminal_1x02
- added J1: Screw_Terminal_1x03, symbol Screw_Terminal_1x03
- renumbered P37 to J2, P4 to J3, P5 to J4, P6 to J5
Connections:
- net GND: now also D1.2 (A), J4.9 (P9), J1.2
- net at J3.14 (P14): no longer D1.2 (A)
- net at F1.2: now also J1.1
- new net GNDPWR: J1.3
Other:
- note added: "+"
- note added: "-"
- note added: "All unit connected to Raspberry Pi via 3 slot GPIO expansion module by J3-5 plugs."
- note added: "PE"
- note added: "Power in\n(5V 2.5A DC)"
- note removed: "Power in"
Changed lines of the file:
@@
 $EndDescr
 $Comp
-L DB9 P37
+L DB9 J2
 U 1 1 5D59B75A
 P 2050 1200
-F 0 "P37" V 2100 1800 50  0000 C CNN
+F 0 "J2" V 2100 1800 50  0000 C CNN
 F 1 "DB9" H 2050 650 50  0001 C CNN
 F 2 "" H 2050 1200 50  0000 C CNN
@@
 $EndComp
 $Comp
-L CONN_02X20 P5
+L CONN_02X20 J4
 U 1 1 5E3076A1
 P 5750 3500
-F 0 "P5" H 5750 4550 50  0000 C CNN
+F 0 "J4" H 5750 4550 50  0000 C CNN
 F 1 "CONN_02X20" V 5750 3500 50  0001 C CNN
 F 2 "" H 5750 2550 50  0000 C CNN
@@
 $EndComp
 $Comp
-L CONN_02X20 P4
+L CONN_02X20 J3
 U 1 1 5E3088F3
 P 2300 3500
-F 0 "P4" H 2300 4550 50  0000 C CNN
+F 0 "J3" H 2300 4550 50  0000 C CNN
 F 1 "CONN_02X20" V 2300 3500 50  0001 C CNN
 F 2 "" H 2300 2550 50  0000 C CNN
@@
 $EndComp
 $Comp
-L CONN_02X20 P6
+L CONN_02X20 J5
 U 1 1 5E3094F6
 P 9650 3500
-F 0 "P6" H 9650 4550 50  0000 C CNN
+F 0 "J5" H 9650 4550 50  0000 C CNN
 F 1 "CONN_02X20" V 9650 3500 50  0001 C CNN
 F 2 "" H 9650 2550 50  0000 C CNN
@@
 Text Label 6200 6250 1    60   ~ 0
 GPIO25
-Text Label 6400 6250 1    60   ~ 0
-+5V
 Text Label 6300 6250 1    60   ~ 0
 GPIO26
+Text Label 6400 6250 1    60   ~ 0
++3.3V
 Text Label 6500 6250 1    60   ~ 0
-+3.3V
-Text Label 6600 6250 1    60   ~ 0
 GND
 Text Label 5450 3150 2    60   ~ 0
@@
 NoConn ~ 5500 2750
 NoConn ~ 5500 2850
-NoConn ~ 5500 2950
 NoConn ~ 5500 3050
 NoConn ~ 5500 3550
@@
 NoConn ~ 6000 2950
 NoConn ~ 6000 3050
-NoConn ~ 6000 3150
 Text Label 6050 4450 0    60   ~ 0
 GPIO21
@@
 Text Label 6050 3250 0    60   ~ 0
 GPIO23
-Text Label 6050 2650 0    60   ~ 0
-+5V
 Text Label 6050 2750 0    60   ~ 0
 GND
@@
 	5200 5650 5200 6300
 Wire Wire Line
-	6400 6300 6400 5750
-Wire Wire Line
-	6400 5750 7200 5750
-Wire Wire Line
-	7200 5750 7200 2650
-Wire Wire Line
-	7200 2650 6000 2650
-Wire Wire Line
 	6000 2750 7300 2750
 Wire Wire Line
 	7300 2750 7300 5850
 Wire Wire Line
-	7300 5850 6600 5850
-Wire Wire Line
-	6600 5850 6600 6300
-Wire Wire Line
-	6500 6300 6500 5850
-Wire Wire Line
-	6500 5850 4900 5850
+	7300 5850 6500 5850
+Wire Wire Line
+	6500 5850 6500 6300
+Wire Wire Line
+	6400 6300 6400 5850
+Wire Wire Line
+	6400 5850 4900 5850
 Wire Wire Line
 	4900 5850 4900 5250
@@
 	9100 2200 9100 2100
 Wire Wire Line
-	6300 6300 6300 5750
-Wire Wire Line
-	6300 5750 3350 5750
+	6300 5750 6300 6300
+Wire Wire Line
+	1500 5750 6300 5750
 Wire Wire Line
 	1500 5750 1500 4350
@@
 	2900 3350 2900 5150
 $Sheet
-S 4900 6300 1750 650
+S 4900 6300 1700 650
 U 5D5B105C
 F0 "U4" 60
 F1 "u4.sch" 60
-F2 "VCC5" I T 6400 6300 60
-F3 "GND" U T 6600 6300 60
-F4 "LED1" I T 5000 6300 60
-F5 "LED2" I T 5100 6300 60
-F6 "LED3" I T 5200 6300 60
-F7 "LED4" I T 5300 6300 60
-F8 "LED5" I T 5400 6300 60
-F9 "LED6" I T 5500 6300 60
-F10 "LED7" I T 5600 6300 60
-F11 "LED8" I T 5700 6300 60
-F12 "LED9" I T 5800 6300 60
-F13 "LED10" I T 5900 6300 60
-F14 "LED11" I T 6000 6300 60
-F15 "LED12" I T 6100 6300 60
-F16 "LED13" I T 6200 6300 60
-F17 "VCC3" I T 6500 6300 60
-F18 "SW" O T 6300 6300 60
+F2 "GND" U T 6500 6300 60
+F3 "LED1" I T 5000 6300 60
+F4 "LED2" I T 5100 6300 60
+F5 "LED3" I T 5200 6300 60
+F6 "LED4" I T 5300 6300 60
+F7 "LED5" I T 5400 6300 60
+F8 "LED6" I T 5500 6300 60
+F9 "LED7" I T 5600 6300 60
+F10 "LED8" I T 5700 6300 60
+F11 "LED9" I T 5800 6300 60
+F12 "LED10" I T 5900 6300 60
+F13 "LED11" I T 6000 6300 60
+F14 "LED12" I T 6100 6300 60
+F15 "LED13" I T 6200 6300 60
+F16 "VCC3" I T 6400 6300 60
+F17 "SW" O T 6300 6300 60
 $EndSheet
 Text Notes 2250 6800 0    60   ~ 0
@@
 Text Notes 5300 950  0    60   ~ 0
 Matrix display
-$Comp
-L Screw_Terminal_1x02 J1
-U 1 1 5E3247FA
-P 3800 6900
-F 0 "J1" V 3800 7150 50  0000 C TNN
-F 1 "Screw_Terminal_1x02" V 3650 6900 50  0001 C TNN
-F 2 "" H 3800 6675 50  0001 C CNN
-F 3 "" H 3775 6900 50  0001 C CNN
-	1    3800 6900
-	0    -1   -1   0
-$EndComp
 Wire Wire Line
 	3700 6700 3700 6650
-Wire Wire Line
-	3700 2550 3700 6200
-Wire Wire Line
-	3700 6200 3700 6350
-Wire Wire Line
-	3700 2550 2950 2550
-Wire Wire Line
-	2950 2550 2550 2550
 Text Label 2600 2550 0    60   ~ 0
 +5V
 Wire Wire Line
-	2550 3150 3900 3150
-Wire Wire Line
-	3900 3150 3900 5650
-Wire Wire Line
-	3900 5650 3900 6700
+	3900 2950 3900 6700
 Wire Wire Line
 	3500 6100 3500 6200
@@
 	3500 5650 3900 5650
 Connection ~ 3900 5650
-Text Notes 3600 7100 0    60   ~ 0
-Power in
+Text Notes 3575 7275 0    60   ~ 0
+  Power in\n(5V 2.5A DC)
 Wire Wire Line
 	1750 1650 1750 2150
@@
 Wire Wire Line
 	2950 2150 2950 2550
-Connection ~ 2950 2550
 Text Label 2600 2650 0    60   ~ 0
 +5V
@@
 +5V
 Wire Wire Line
-	3350 5750 1500 5750
+	2950 2550 2550 2550
+Wire Wire Line
+	3700 2350 3700 6350
+Wire Wire Line
+	3700 2350 6450 2350
+Wire Wire Line
+	6450 2350 6450 2650
+Wire Wire Line
+	6450 2650 6000 2650
+Wire Wire Line
+	5500 2950 3900 2950
+Text Label 5450 2950 2    60   ~ 0
+GND
+Text Label 6050 2650 0    60   ~ 0
++5V
+NoConn ~ 6000 3150
+NoConn ~ 2550 3150
+Text Notes 3675 7050 0    60   ~ 0
++
+$Comp
+L Screw_Terminal_1x03 J1
+U 1 1 5E3366A9
+P 3900 6900
+F 0 "J1" V 3900 6550 50  0000 C TNN
+F 1 "Screw_Terminal_1x03" V 3750 6900 50  0001 C TNN
+F 2 "" H 3900 6575 50  0001 C CNN
+F 3 "" H 3875 7000 50  0001 C CNN
+	1    3900 6900
+	0    -1   -1   0
+$EndComp
+Text Notes 3875 7050 0    60   ~ 0
+-
+Text Notes 4050 7075 0    60   ~ 0
+PE
+$Comp
+L GNDPWR #PWR01
+U 1 1 5E336A2A
+P 4425 6750
+F 0 "#PWR01" H 4425 6550 50  0001 C CNN
+F 1 "GNDPWR" H 4425 6620 50  0001 C CNN
+F 2 "" H 4425 6700 50  0000 C CNN
+F 3 "" H 4425 6700 50  0000 C CNN
+	1    4425 6750
+	1    0    0    -1
+$EndComp
+Wire Wire Line
+	4100 6700 4100 6600
+Wire Wire Line
+	4100 6600 4425 6600
+Wire Wire Line
+	4425 6600 4425 6750
+Text Notes 7150 6300 0    60   ~ 0
+All unit connected to Raspberry Pi via 3 slot GPIO expansion module by J3-5 plugs.
 $EndSCHEMATC

Commit message: 200213
Parts:
- added C1: 1000u, symbol CP
- added C2, C3: 100n, symbol C
- added C4: 4.7u, symbol CP
- added L1: L_Core_Ferrite, symbol L_Core_Ferrite
- added LS1: 8 ohm 0.3 W, symbol Speaker
- added R1: 270, symbol R
- added R2: 150, symbol R
- added R3: 15k, symbol R
- added R4: 10, symbol R
- added SW1: SWITCH_1P, symbol SWITCH_1P
- added T1: 2N2222, symbol Q_NPN_EBC
- J2: value DB9 -> DB9 female
Connections:
- net +5V: now also C1.1, C2.2, L1.2, LS1.1, R3.2, SW1.2; no longer D1.1 (K), F1.1
- net GND: now also C1.2, C2.1, C3.2, R2.1, T1.1 (E)
- net GPIO17: now reaches J5.11 (P11)
- net GPIO17: now also R1.1
- new net: D1.1 (K), F1.1, L1.1
- new net: C3.1, C4.2, R1.2, R2.2
- new net: C4.1, R3.1, T1.2 (B)
- new net: LS1.2, R4.1
- new net: R4.2, T1.3 (C)
- new net +5V-Relay: SW1.1, U6.~ (VCCJb), U7.~ (VCCJb)
- no-connect marks 75 -> 76
Other:
- note added: "Disable outputs\n (key switch)"
- moved on the sheet: U7
