File: cad_files/mm5d/u3.sch (KiCad schematic (older format))
At the start: 0 parts

Commit message: 190922
Parts:
- added C301, C302: 4.7u, symbol CP
- added D301, D302, D303, D304: 1N4001, symbol D
- added F301: 100 mA F, symbol Fuse
- added R301, R302, R303, R304: 10, symbol R
- added R305, R306, R307, R308: 1k, symbol R
- added U301, U302: Level_shifter_4, symbol Level_shifter_4
Connections:
- net +5V: now also C302.1, F301.2, U301.~ (LV4), U302.~ (LV4)
- net DATA_S1: now also U301.~ (LV4)
- net DATA_S2: now also U301.~ (LV4)
- net GND: now also C301.2, C302.2, D301.2 (A), D302.2 (A), D303.2 (A), D304.2 (A), U301.~ (LV4), U302.~ (LV4)
- net LED1: now also D301.1 (K), R301.1, R305.2, U302.~ (LV4)
- net LED2: now also D302.1 (K), R302.1, R306.2, U302.~ (LV4)
- net LED3: now also D303.1 (K), R303.1, R307.2, U302.~ (LV4)
- net LED4: now also D304.1 (K), R304.1, R308.2, U302.~ (LV4)
- net OUT1: now also U302.~ (LV4)
- net OUT2: now also U302.~ (LV4)
- net OUT3: now also U302.~ (LV4)
- net OUT4: now also U302.~ (LV4)
- new net: R305.1, R306.1, R307.1, R308.1
- new net +3V3: C301.1, U301.~ (LV4), U302.~ (LV4)
- new net +5V-S: F301.1
- new net DATA-S1: U301.~ (LV4)
- new net DATA-S2: U301.~ (LV4)
- new net IN1: R301.2
- new net IN2: R302.2
- new net IN3: R303.2
- new net IN4: R304.2
- no-connect marks 0 -> 4

Commit message: 190922
Changed lines of the file:
@@
 	1200 7825 1500 7825
 Wire Wire Line
-	1500 7625 1500 7825
-Wire Wire Line
-	1500 7825 1500 7875
+	1500 7625 1500 7875
 Wire Wire Line
 	1200 7725 1900 7725
 Wire Wire Line
-	1900 7625 1900 7725
+	1900 7625 1900 7875
 Wire Wire Line
-	1900 7725 1900 7875
+	1200 8225 1900 8225
 Wire Wire Line
-	1200 8225 1500 8225
-Wire Wire Line
-	1500 8225 1900 8225
-Wire Wire Line
-	1900 8175 1900 8225
-Wire Wire Line
-	1900 8225 1900 8275
+	1900 8175 1900 8275
 Wire Wire Line
 	1500 8175 1500 8225
@@
 Connection ~ 1500 7825
 Wire Wire Line
-	1800 2725 2025 2725
+	1800 2725 7100 2725
 Wire Wire Line
-	2025 2725 5800 2725
+	1800 2875 7100 2875
 Wire Wire Line
-	5800 2725 7100 2725
+	1800 3025 7100 3025
 Wire Wire Line
-	1800 2875 2325 2875
+	1800 3175 7100 3175
 Wire Wire Line
-	2325 2875 5900 2875
+	2025 2425 2025 3425
 Wire Wire Line
-	5900 2875 7100 2875
+	2325 2425 2325 3425
 Wire Wire Line
-	1800 3025 2625 3025
+	2625 2425 2625 3425
 Wire Wire Line
-	2625 3025 6000 3025
-Wire Wire Line
-	6000 3025 7100 3025
-Wire Wire Line
-	1800 3175 2925 3175
-Wire Wire Line
-	2925 3175 6100 3175
-Wire Wire Line
-	6100 3175 7100 3175
-Wire Wire Line
-	2025 2425 2025 2725
-Wire Wire Line
-	2025 2725 2025 3425
-Wire Wire Line
-	2325 2425 2325 2875
-Wire Wire Line
-	2325 2875 2325 3425
-Wire Wire Line
-	2625 2425 2625 3025
-Wire Wire Line
-	2625 3025 2625 3425
-Wire Wire Line
-	2925 2425 2925 3175
-Wire Wire Line
-	2925 3175 2925 3425
+	2925 2425 2925 3425
 Connection ~ 2025 2725
 Connection ~ 2325 2875
@@
 	2025 3725 2025 3825
 Wire Wire Line
-	1350 3825 2025 3825
-Wire Wire Line
-	2025 3825 2325 3825
-Wire Wire Line
-	2325 3825 2625 3825
-Wire Wire Line
-	2625 3825 2925 3825
-Wire Wire Line
-	2925 3825 4325 3825
-Wire Wire Line
-	4325 3825 5700 3825
+	1350 3825 5700 3825
 Wire Wire Line
 	2925 3825 2925 3725
@@
 	2025 2125 2025 2025
 Wire Wire Line
-	2025 2025 2325 2025
-Wire Wire Line
-	2325 2025 2625 2025
-Wire Wire Line
-	2625 2025 2925 2025
+	2025 2025 2925 2025
 Wire Wire Line
 	2925 2025 2925 2125
@@
 	1200 3325 1350 3325
 Wire Wire Line
-	1350 3325 1350 3825
-Wire Wire Line
-	1350 3825 1350 4325
+	1350 3325 1350 4325
 Connection ~ 2025 3825
 Wire Wire Line
@@
 Connection ~ 6100 3175
 Wire Wire Line
-	5700 3825 5700 5575
-Wire Wire Line
-	5700 5575 5700 5775
+	5700 3825 5700 5775
 Connection ~ 2925 3825
 Wire Wire Line
-	6200 5350 6200 5475
+	6200 5350 6200 5775
 Wire Wire Line
-	6200 5475 6200 5775
-Wire Wire Line
-	6200 7075 6200 7375
-Wire Wire Line
-	6200 7375 6200 7475
+	6200 7075 6200 7475
 Wire Wire Line
 	5800 7075 5800 7775
@@
 	4275 4625 4275 5775
 Wire Wire Line
-	4075 5575 5050 5575
-Wire Wire Line
-	5050 5575 5700 5575
+	4075 5575 5700 5575
 Wire Wire Line
 	4075 5575 4075 5775
@@
 	5700 7275 5700 7075
 Wire Wire Line
-	4075 7275 5050 7275
-Wire Wire Line
-	5050 7275 5700 7275
+	4075 7275 5700 7275
 Wire Wire Line
 	4075 7275 4075 7075
