File: cad_files/mm5d/u3.sch (KiCad schematic (older format))
At the start: 17 parts, among them U301 Level_shifter_4, U302 Level_shifter_4

Commit message: 191005
Parts:
- R301, R302, R303, R304: value 10 -> 100
Changed lines of the file:
@@
 U 1 1 5D881151
 P 1650 2725
-F 0 "R301" V 1550 2500 50  0000 C CNN
-F 1 "10" V 1725 2925 50  0000 C CNN
+F 0 "R301" V 1575 2500 50  0000 C CNN
+F 1 "100" V 1725 2925 50  0000 C CNN
 F 2 "" V 1580 2725 50  0000 C CNN
 F 3 "" H 1650 2725 50  0000 C CNN
@@
 P 1650 2875
 F 0 "R302" V 1575 2650 50  0000 C CNN
-F 1 "10" V 1725 3075 50  0000 C CNN
+F 1 "100" V 1725 3075 50  0000 C CNN
 F 2 "" V 1580 2875 50  0000 C CNN
 F 3 "" H 1650 2875 50  0000 C CNN
@@
 P 1650 3025
 F 0 "R303" V 1575 2800 50  0000 C CNN
-F 1 "10" V 1725 3225 50  0000 C CNN
+F 1 "100" V 1725 3225 50  0000 C CNN
 F 2 "" V 1580 3025 50  0000 C CNN
 F 3 "" H 1650 3025 50  0000 C CNN
@@
 P 1650 3175
 F 0 "R304" V 1575 2950 50  0000 C CNN
-F 1 "10" V 1725 3375 50  0000 C CNN
+F 1 "100" V 1725 3375 50  0000 C CNN
 F 2 "" V 1580 3175 50  0000 C CNN
 F 3 "" H 1650 3175 50  0000 C CNN
