File: cad_files/mm5d/u2.sch (KiCad schematic (older format))
At the start: 0 parts

Commit message: 190922
Parts:
- added P?: CONN_02X20, symbol CONN_02X20
Connections:
- net CE0: now also P?.24 (P24)
- net GPIO12: now also P?.32 (P32)
- net GPIO13: now also P?.33 (P33)
- net GPIO16: now also P?.36 (P36)
- net GPIO17: now also P?.11 (P11)
- net GPIO18: now also P?.12 (P12)
- net GPIO19: now also P?.35 (P35)
- net GPIO2: now also P?.3 (P3)
- net GPIO20: now also P?.38 (P38)
- net GPIO21: now also P?.40 (P40)
- net GPIO22: now also P?.15 (P15)
- net GPIO23: now also P?.16 (P16)
- net GPIO24: now also P?.18 (P18)
- net GPIO25: now also P?.22 (P22)
- net GPIO26: now also P?.37 (P37)
- net GPIO27: now also P?.13 (P13)
- net GPIO3: now also P?.5 (P5)
- net GPIO4: now also P?.7 (P7)
- net GPIO5: now also P?.29 (P29)
- net GPIO6: now also P?.31 (P31)
- net MOSI: now also P?.19 (P19)
- net SCLK: now also P?.23 (P23)
- new net: P?.2 (P2), P?.4 (P4)
Changed lines of the file:
@@
 EELAYER 25 0
 EELAYER END
-$Descr A4 11693 8268
+$Descr A4 8268 11693 portrait
 encoding utf-8
 Sheet 3 4
@@
 Comment4 ""
 $EndDescr
-Text HLabel 1750 1300 0    60   BiDi ~ 0
+Text HLabel 1300 4000 0    60   Output ~ 0
 GPIO2
-Text HLabel 1750 1400 0    60   BiDi ~ 0
+Text HLabel 1300 4100 0    60   Output ~ 0
 GPIO3
-Text HLabel 1750 1500 0    60   BiDi ~ 0
+Text HLabel 1300 4200 0    60   Output ~ 0
 GPIO4
-Text HLabel 1750 1600 0    60   BiDi ~ 0
+Text HLabel 1300 4300 0    60   Output ~ 0
 GPIO5
-Text HLabel 1750 1700 0    60   BiDi ~ 0
+Text HLabel 1300 4400 0    60   Output ~ 0
 GPIO6
-Text HLabel 1750 1800 0    60   BiDi ~ 0
+Text HLabel 1300 4500 0    60   Output ~ 0
 GPIO12
-Text HLabel 1750 1900 0    60   BiDi ~ 0
+Text HLabel 1300 4600 0    60   Output ~ 0
 GPIO13
-Text HLabel 1750 2000 0    60   BiDi ~ 0
-TXD
-Text HLabel 1750 2100 0    60   BiDi ~ 0
-RXD
-Text HLabel 1750 2200 0    60   BiDi ~ 0
+Text HLabel 1300 4700 0    60   Output ~ 0
 GPIO16
-Text HLabel 1750 2300 0    60   BiDi ~ 0
+Text HLabel 1300 4800 0    60   BiDi ~ 0
 GPIO17
-Text HLabel 1750 2400 0    60   BiDi ~ 0
+Text HLabel 1300 4900 0    60   BiDi ~ 0
 GPIO18
-Text HLabel 1750 2500 0    60   BiDi ~ 0
+Text HLabel 1300 5000 0    60   Output ~ 0
 GPIO19
-Text HLabel 1750 2600 0    60   BiDi ~ 0
+Text HLabel 1300 5100 0    60   Output ~ 0
 GPIO20
-Text HLabel 1750 2700 0    60   BiDi ~ 0
+Text HLabel 1300 5200 0    60   Output ~ 0
 GPIO21
-Text HLabel 1750 2800 0    60   BiDi ~ 0
+Text HLabel 1300 5300 0    60   Input ~ 0
 GPIO22
-Text HLabel 1750 2900 0    60   BiDi ~ 0
+Text HLabel 1300 5400 0    60   Input ~ 0
 GPIO23
-Text HLabel 1750 3000 0    60   BiDi ~ 0
+Text HLabel 1300 5500 0    60   Input ~ 0
 GPIO24
-Text HLabel 1750 3100 0    60   BiDi ~ 0
+Text HLabel 1300 5600 0    60   Output ~ 0
 GPIO25
-Text HLabel 1750 3200 0    60   BiDi ~ 0
+Text HLabel 1300 5700 0    60   BiDi ~ 0
 GPIO26
-Text HLabel 1750 3300 0    60   BiDi ~ 0
+Text HLabel 1300 5800 0    60   Input ~ 0
 GPIO27
-Text HLabel 1750 3400 0    60   BiDi ~ 0
+Text HLabel 7050 975  2    60   BiDi ~ 0
 MOSI
-Text HLabel 1750 3500 0    60   Output ~ 0
+Text HLabel 7050 1075 2    60   Output ~ 0
 CE0
-Text HLabel 1750 3600 0    60   Output ~ 0
+Text HLabel 7050 1175 2    60   Output ~ 0
 SCLK
-Text HLabel 2300 1300 0    60   Output ~ 0
-+5V
-Text HLabel 2300 1400 0    60   UnSpc ~ 0
-GND
-Text HLabel 2750 1750 0    60   Output ~ 0
-LED1
-Text HLabel 2750 1950 0    60   Output ~ 0
-LED2
-Text HLabel 2700 2200 0    60   Output ~ 0
-LED3
-Text HLabel 2700 2500 0    60   Output ~ 0
-LED4
+$Comp
+L CONN_02X20 P?
+U 1 1 5D87E6B0
+P 3725 3500
+F 0 "P?" H 3725 4550 50  0000 C CNN
+F 1 "CONN_02X20" V 3725 3500 50  0000 C CNN
+F 2 "" H 3725 2550 50  0000 C CNN
+F 3 "" H 3725 2550 50  0000 C CNN
+	1    3725 3500
+	0    -1   -1   0
+$EndComp
+Text HLabel 7050 4300 2    60   Output ~ 0
+GPIO5'
+Text HLabel 7050 4400 2    60   Output ~ 0
+GPIO6'
+Text HLabel 7050 4600 2    60   Output ~ 0
+GPIO13'
+Text HLabel 7050 5000 2    60   Output ~ 0
+GPIO19'
+Wire Wire Line
+	2875 3175 2875 3250
+Wire Wire Line
+	2775 3175 2875 3175
+Wire Wire Line
+	2775 3250 2775 3175
+Wire Wire Line
+	3875 4800 3875 3750
+Wire Wire Line
+	6850 4800 3875 4800
+Wire Wire Line
+	6850 1175 6850 4800
+Wire Wire Line
+	7050 1175 6850 1175
+Wire Wire Line
+	6750 975  7050 975
+Wire Wire Line
+	6750 4200 6750 975
+Wire Wire Line
+	3675 4200 6750 4200
+Wire Wire Line
+	3675 3750 3675 4200
+Wire Wire Line
+	3875 1075 7050 1075
+Wire Wire Line
+	3875 3250 3875 1075
+Connection ~ 4475 5000
+Connection ~ 4375 4600
+Connection ~ 4275 4400
+Connection ~ 4175 4300
+Wire Wire Line
+	3775 2675 3775 3250
+Wire Wire Line
+	2475 2675 3775 2675
+Wire Wire Line
+	2475 5600 2475 2675
+Wire Wire Line
+	1300 5600 2475 5600
+Wire Wire Line
+	2375 5500 1300 5500
+Wire Wire Line
+	2375 2775 2375 5500
+Wire Wire Line
+	3575 2775 2375 2775
+Wire Wire Line
+	3575 3250 3575 2775
+Wire Wire Line
+	3475 2875 3475 3250
+Wire Wire Line
+	2275 2875 3475 2875
+Wire Wire Line
+	2275 5400 2275 2875
+Wire Wire Line
+	1300 5400 2275 5400
+Wire Wire Line
+	4675 2975 4675 3250
+Wire Wire Line
+	5925 2975 4675 2975
+Wire Wire Line
+	5925 5200 5925 2975
+Wire Wire Line
+	1300 5200 5925 5200
+Wire Wire Line
+	4575 2875 4575 3250
+Wire Wire Line
+	5825 2875 4575 2875
+Wire Wire Line
+	5825 5100 5825 2875
+Wire Wire Line
+	1300 5100 5825 5100
+Wire Wire Line
+	3275 2975 3275 3250
+Wire Wire Line
+	2175 2975 3275 2975
+Wire Wire Line
+	2175 4900 2175 2975
+Wire Wire Line
+	1300 4900 2175 4900
+Wire Wire Line
+	4475 2775 4475 3250
+Wire Wire Line
+	5625 2775 4475 2775
+Wire Wire Line
+	5625 4700 5625 2775
+Wire Wire Line
+	1300 4700 5625 4700
+Wire Wire Line
+	4275 2675 4275 3250
+Wire Wire Line
+	5450 2675 4275 2675
+Wire Wire Line
+	5450 4500 5450 2675
+Wire Wire Line
+	1300 4500 5450 4500
+Wire Wire Line
+	3375 5800 3375 3750
+Wire Wire Line
+	1300 5800 3375 5800
+Wire Wire Line
+	4575 5700 4575 3750
+Wire Wire Line
+	1300 5700 4575 5700
+Wire Wire Line
+	3475 5300 3475 3750
+Wire Wire Line
+	1300 5300 3475 5300
+Wire Wire Line
+	4475 5000 7050 5000
+Wire Wire Line
+	1300 5000 4475 5000
+Wire Wire Line
+	4475 3750 4475 5000
+Wire Wire Line
+	3275 4800 3275 3750
+Wire Wire Line
+	1300 4800 3275 4800
+Wire Wire Line
+	4375 4600 7050 4600
+Wire Wire Line
+	1300 4600 4375 4600
+Wire Wire Line
+	4375 3750 4375 4600
+Wire Wire Line
+	4275 4400 4275 3750
+Wire Wire Line
+	4275 4400 7050 4400
+Wire Wire Line
+	1300 4400 4275 4400
+Wire Wire Line
+	4175 4300 4175 3750
+Wire Wire Line
+	4175 4300 7050 4300
+Wire Wire Line
+	1300 4300 4175 4300
+Wire Wire Line
+	3075 4200 3075 3750
+Wire Wire Line
+	1300 4200 3075 4200
+Wire Wire Line
+	2975 4100 2975 3750
+Wire Wire Line
+	1300 4100 2975 4100
+Wire Wire Line
+	2875 4000 2875 3750
+Wire Wire Line
+	1300 4000 2875 4000
 $EndSCHEMATC

Commit message: 190922
Parts:
- added C201: 100u, symbol CP
- added C202, C203, C204, C205, C206: 100n, symbol C
- added JP201, JP? (x6): Jumper_NO_Small, symbol Jumper_NO_Small
- added U201: MAX3232CPE, symbol MAX232
- gave numbers to parts that had none: 1
Connections:
- net GPIO13: now also JP?.1
- net GPIO19: now also JP?.1
- net GPIO2: now also JP?.1
- net GPIO3: now also JP?.1
- net GPIO4: now also JP?.1
- net GPIO5: now also JP201.1
- net GPIO6: now also JP?.1
- net +3.3V-1: now reaches P201.1 (P1)
- net +3.3V-1: now also P201.17 (P17), C202.1, U201.16 (VCC)
- net at P201.10 (P10): now also U201.12 (R1OUT)
- net GND: now reaches P201.14 (P14)
- net GND: now also P201.20 (P20), P201.25 (P25), P201.30 (P30), P201.34 (P34), P201.39 (P39), P201.6 (P6), P201.9 (P9), C201.2, C202.2, C205.2, C206.2, U201.15 (GND)
- net +5V: now reaches P201.2 (P2), P201.4 (P4)
- net +5V: now also C201.1
- net at P201.8 (P8): now also U201.11 (T1IN)
- new net: C203.1, U201.1 (C1+)
- new net: C205.1, U201.2 (VS+)
- new net: C203.2, U201.3 (C1-)
- new net: C204.1, U201.4 (C2+)
- new net: C204.2, U201.5 (C2-)
- new net: C206.1, U201.6 (VS-)
- new net OUT8: JP201.2, JP?.2, JP?.2, JP?.2, JP?.2, JP?.2, JP?.2
- new net RXD: U201.13 (R1IN)
- new net TXD: U201.14 (T1OUT)
- no-connect marks 0 -> 4
Other:
- note added: "Connector for the Rasperry Pi GPIO port"
- moved on the sheet: P201
