File: cad_files/mm5d/u2.sch (KiCad schematic (older format))
At the start: 15 parts, among them P201 CONN_02X20, U201 MAX3232CPE

Commit message: 191005
Connections:
- net +3.3V-1 is gone; now on net GND: C202.1, P201.1 (P1), P201.17 (P17), U201.16 (VCC)
Other:
- note added: "P202"
- note added: "P203"
- note added: "P204"
- moved on the sheet: C201
