File: cad_files/mm5d/u6.sch (KiCad schematic (older format))
At the start: 30 parts

Commit message: 190920
Parts:
- added P602: CONN_01X05, symbol CONN_01X05
- gave numbers to parts that had none: 27
- renumbered R601 to R602
Connections:
- net +3.3V is gone; now on net +3V3: C601.1
- net +3V3: no longer C602.1, D601.2 (A), D602.2 (A), D603.2 (A), D604.2 (A), D605.2 (A)
- net CLK: now also P602.5 (P5)
- net CS: now also P602.4 (P4)
- net DIN: now also P602.3 (P3)
- net GND: now also P602.2 (P2)
- new net +5V: C602.1, D601.2 (A), D602.2 (A), D603.2 (A), D604.2 (A), D605.2 (A), P602.1 (P1)
Other:
- note added: "ERR1"
- note added: "ERR2"
- note added: "ERR3"
- note added: "ERR4"
- note added: "OUT1"
- note added: "OUT2"
- note added: "OUT3"
- note added: "OUT4"
- note added: "P601"
- note added: "connector of 4 pcs 8x8\nmatrix display modul"
- moved on the sheet: C602, D601, D602, D603, D604, D605, D606, D607, D608, D609, D610, D611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

Commit message: 190920
Connections:
- net CLK renamed SCLK
- net CS renamed CE0
- net DIN renamed MOSI
Changed lines of the file:
@@
 LIBS:contrib
 LIBS:valves
+LIBS:pozsarzs
 LIBS:mm5d-cache
 EELAYER 25 0
@@
 $Descr A4 11693 8268
 encoding utf-8
-Sheet 6 6
+Sheet 4 4
 Title "MM5D controlling and remote monitoring equipment"
 Date "2019-09-15"
@@
 GND
 Text HLabel 1200 5275 0    60   Input ~ 0
-DIN
+MOSI
 Text HLabel 1200 5375 0    60   Input ~ 0
-CS
+CE0
 Text HLabel 1200 5475 0    60   Input ~ 0
-CLK
+SCLK
 Text HLabel 1200 2825 0    60   Input ~ 0
 LED1

Commit message: 190922
Other:
- note added: "connector of 32x8 matrix display modul"
- note removed: "connector of 4 pcs 8x8\nmatrix display modul"
- moved on the sheet: C601, C602, D601, D602, D603, D604, D605, D606, D607, D608, D609, D610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

Commit message: 190922
Other:
- note removed: "P601"
Changed lines of the file:
@@
 	1350 7775 1650 7775
 Wire Wire Line
-	1650 7575 1650 7775
-Wire Wire Line
-	1650 7775 1650 7825
+	1650 7575 1650 7825
 Wire Wire Line
 	1350 7675 2050 7675
 Wire Wire Line
-	2050 7575 2050 7675
-Wire Wire Line
-	2050 7675 2050 7825
-Wire Wire Line
-	1350 8175 1650 8175
-Wire Wire Line
-	1650 8175 2050 8175
-Wire Wire Line
-	2050 8125 2050 8175
-Wire Wire Line
-	2050 8175 2050 8225
+	2050 7575 2050 7825
+Wire Wire Line
+	1350 8175 2050 8175
+Wire Wire Line
+	2050 8125 2050 8225
 Wire Wire Line
 	1650 8125 1650 8175
@@
 	2550 2700 2550 2600
 Wire Wire Line
-	2100 2600 2550 2600
-Wire Wire Line
-	2550 2600 2850 2600
-Wire Wire Line
-	2850 2600 3150 2600
-Wire Wire Line
-	3150 2600 3450 2600
-Wire Wire Line
-	3450 2500 3450 2600
-Wire Wire Line
-	3450 2600 3450 2700
+	2100 2600 3450 2600
+Wire Wire Line
+	3450 2500 3450 2700
 Wire Wire Line
 	3900 2700 3900 2600
 Wire Wire Line
-	3900 2600 4200 2600
-Wire Wire Line
-	4200 2600 4500 2600
-Wire Wire Line
-	4500 2600 4800 2600
-Wire Wire Line
-	4800 2600 5300 2600
-Wire Wire Line
-	5300 2600 5600 2600
-Wire Wire Line
-	5600 2600 5900 2600
-Wire Wire Line
-	5900 2600 6200 2600
-Wire Wire Line
-	6200 2500 6200 2600
-Wire Wire Line
-	6200 2600 6200 2700
+	3900 2600 6200 2600
+Wire Wire Line
+	6200 2500 6200 2700
 Wire Wire Line
 	2850 2700 2850 2600
@@
 Text Notes 2550 6300 0    60   ~ 0
 connector of 32x8 matrix display modul
-Text Notes 1100 3625 0    60   ~ 0
-P601
 $EndSCHEMATC

Commit message: 190923
Parts:
- added R615: 1k, symbol R
- added SW601: SWITCH_1P, symbol SWITCH_1P
Connections:
- net +3V3: now also R615.2
- net GND: now also SW601.2
- new net SW-MODE: R615.1, SW601.1
Other:
- note added: "MODE"
- moved on the sheet: P602
Changed lines of the file:
@@
 Text HLabel 1350 8175 0    60   UnSpc ~ 0
 GND
-Text HLabel 1350 6250 0    60   Input ~ 0
+Text HLabel 1350 6725 0    60   Input ~ 0
 MOSI
-Text HLabel 1350 6350 0    60   Input ~ 0
+Text HLabel 1350 6825 0    60   Input ~ 0
 CE0
-Text HLabel 1350 6450 0    60   Input ~ 0
+Text HLabel 1350 6925 0    60   Input ~ 0
 SCLK
 Text HLabel 1350 3800 0    60   Input ~ 0
@@
 P 1650 7575
 F 0 "#PWR601" H 1650 7425 50  0001 C CNN
-F 1 "+3.3V" H 1650 7715 50  0000 C CNN
+F 1 "+3.3V" H 1650 7750 50  0000 C CNN
 F 2 "" H 1650 7575 50  0000 C CNN
 F 3 "" H 1650 7575 50  0000 C CNN
@@
 P 2050 7575
 F 0 "#PWR602" H 2050 7425 50  0001 C CNN
-F 1 "+5V" H 2050 7715 50  0000 C CNN
+F 1 "+5V" H 2050 7750 50  0000 C CNN
 F 2 "" H 2050 7575 50  0000 C CNN
 F 3 "" H 2050 7575 50  0000 C CNN
@@
 P 6200 2500
 F 0 "#PWR606" H 6200 2350 50  0001 C CNN
-F 1 "+3.3V" H 6200 2640 50  0000 C CNN
+F 1 "+3.3V" H 6200 2675 50  0000 C CNN
 F 2 "" H 6200 2500 50  0000 C CNN
 F 3 "" H 6200 2500 50  0000 C CNN
@@
 P 3450 2500
 F 0 "#PWR605" H 3450 2350 50  0001 C CNN
-F 1 "+5V" H 3450 2640 50  0000 C CNN
+F 1 "+5V" H 3450 2675 50  0000 C CNN
 F 2 "" H 3450 2500 50  0000 C CNN
 F 3 "" H 3450 2500 50  0000 C CNN
@@
 	1    0    0    -1
 $EndComp
-Text Notes 2050 2250 0    60   ~ 0
+Text Notes 2050 2200 0    60   ~ 0
 ON
-Text Notes 2500 2250 0    60   ~ 0
+Text Notes 2500 2200 0    60   ~ 0
 IN1
-Text Notes 2800 2250 0    60   ~ 0
+Text Notes 2800 2200 0    60   ~ 0
 IN2
-Text Notes 3100 2250 0    60   ~ 0
+Text Notes 3100 2200 0    60   ~ 0
 IN3
-Text Notes 3400 2250 0    60   ~ 0
+Text Notes 3400 2200 0    60   ~ 0
 IN4
-Text Notes 5200 2250 0    60   ~ 0
+Text Notes 5200 2200 0    60   ~ 0
 OUT1
-Text Notes 5500 2250 0    60   ~ 0
+Text Notes 5500 2200 0    60   ~ 0
 OUT2
-Text Notes 5800 2250 0    60   ~ 0
+Text Notes 5800 2200 0    60   ~ 0
 OUT3
-Text Notes 6100 2250 0    60   ~ 0
+Text Notes 6100 2200 0    60   ~ 0
 OUT4
-Text Notes 3800 2250 0    60   ~ 0
+Text Notes 3800 2200 0    60   ~ 0
 ERR1
-Text Notes 4100 2250 0    60   ~ 0
+Text Notes 4100 2200 0    60   ~ 0
 ERR2
-Text Notes 4400 2250 0    60   ~ 0
+Text Notes 4400 2200 0    60   ~ 0
 ERR3
-Text Notes 4700 2250 0    60   ~ 0
+Text Notes 4700 2200 0    60   ~ 0
 ERR4
-Text Notes 6650 2250 0    60   ~ 0
+Text Notes 6650 2200 0    60   ~ 0
 ACT
 Connection ~ 1650 7775
@@
 L CONN_01X05 P602
 U 1 1 5D860E7B
-P 2350 6250
-F 0 "P602" H 2350 6550 50  0000 C CNN
-F 1 "CONN_01X05" V 2450 6250 50  0001 C CNN
-F 2 "" H 2350 6250 50  0000 C CNN
-F 3 "" H 2350 6250 50  0000 C CNN
-	1    2350 6250
+P 2350 6725
+F 0 "P602" H 2350 7025 50  0000 C CNN
+F 1 "CONN_01X05" V 2450 6725 50  0001 C CNN
+F 2 "" H 2350 6725 50  0000 C CNN
+F 3 "" H 2350 6725 50  0000 C CNN
+	1    2350 6725
 	1    0    0    -1
 $EndComp
@@
 L +5V #PWR?
 U 1 1 5D86109E
-P 2050 5975
-F 0 "#PWR?" H 2050 5825 50  0001 C CNN
-F 1 "+5V" H 2050 6115 50  0000 C CNN
-F 2 "" H 2050 5975 50  0000 C CNN
-F 3 "" H 2050 5975 50  0000 C CNN
-	1    2050 5975
+P 2050 6450
+F 0 "#PWR?" H 2050 6300 50  0001 C CNN
+F 1 "+5V" H 2050 6625 50  0000 C CNN
+F 2 "" H 2050 6450 50  0000 C CNN
+F 3 "" H 2050 6450 50  0000 C CNN
+	1    2050 6450
 	1    0    0    -1
 $EndComp
@@
 L GND #PWR?
 U 1 1 5D86125B
-P 2050 6525
-F 0 "#PWR?" H 2050 6275 50  0001 C CNN
-F 1 "GND" H 2050 6375 50  0001 C CNN
-F 2 "" H 2050 6525 50  0000 C CNN
-F 3 "" H 2050 6525 50  0000 C CNN
-	1    2050 6525
-	1    0    0    -1
-$EndComp
-Wire Wire Line
-	1350 6450 2150 6450
-Wire Wire Line
-	1350 6350 2150 6350
-Wire Wire Line
-	1350 6250 2150 6250
-Wire Wire Line
-	2050 5975 2050 6050
-Wire Wire Line
-	2050 6050 2150 6050
-Wire Wire Line
-	2150 6150 2050 6150
-Wire Wire Line
-	2050 6150 2050 6525
-Text Notes 2550 6300 0    60   ~ 0
+P 2050 7000
+F 0 "#PWR?" H 2050 6750 50  0001 C CNN
+F 1 "GND" H 2050 6850 50  0001 C CNN
+F 2 "" H 2050 7000 50  0000 C CNN
+F 3 "" H 2050 7000 50  0000 C CNN
+	1    2050 7000
+	1    0    0    -1
+$EndComp
+Wire Wire Line
+	1350 6925 2150 6925
+Wire Wire Line
+	1350 6825 2150 6825
+Wire Wire Line
+	1350 6725 2150 6725
+Wire Wire Line
+	2050 6450 2050 6525
+Wire Wire Line
+	2050 6525 2150 6525
+Wire Wire Line
+	2150 6625 2050 6625
+Wire Wire Line
+	2050 6625 2050 7000
+Text Notes 2550 6775 0    60   ~ 0
 connector of 32x8 matrix display modul
+$Comp
+L SWITCH_1P SW601
+U 1 1 5D89AA8D
+P 1975 6000
+F 0 "SW601" H 1975 5875 50  0000 C CNN
+F 1 "SWITCH_1P" H 1975 5900 70  0001 C CNN
+F 2 "" H 1975 6000 60  0000 C CNN
+F 3 "" H 1975 6000 60  0000 C CNN
+	1    1975 6000
+	1    0    0    -1
+$EndComp
+$Comp
+L R R615
+U 1 1 5D89AB4E
+P 1475 5750
+F 0 "R615" H 1300 5675 50  0000 C CNN
+F 1 "1k" H 1350 5825 50  0000 C CNN
+F 2 "" V 1405 5750 50  0000 C CNN
+F 3 "" H 1475 5750 50  0000 C CNN
+	1    1475 5750
+	-1   0    0    1
+$EndComp
+$Comp
+L +3.3V #PWR?
+U 1 1 5D89AC5D
+P 1475 5500
+F 0 "#PWR?" H 1475 5350 50  0001 C CNN
+F 1 "+3.3V" H 1475 5675 50  0000 C CNN
+F 2 "" H 1475 5500 50  0000 C CNN
+F 3 "" H 1475 5500 50  0000 C CNN
+	1    1475 5500
+	1    0    0    -1
+$EndComp
+Text HLabel 1350 6000 0    60   Input ~ 0
+SW-MODE
+$Comp
+L GND #PWR?
+U 1 1 5D89B4C4
+P 2500 6075
+F 0 "#PWR?" H 2500 5825 50  0001 C CNN
+F 1 "GND" H 2500 5925 50  0001 C CNN
+F 2 "" H 2500 6075 50  0000 C CNN
+F 3 "" H 2500 6075 50  0000 C CNN
+	1    2500 6075
+	1    0    0    -1
+$EndComp
+Wire Wire Line
+	1350 6000 1575 6000
+Wire Wire Line
+	1475 6000 1475 5900
+Connection ~ 1475 6000
+Wire Wire Line
+	1475 5600 1475 5500
+Wire Wire Line
+	2425 6000 2500 6000
+Wire Wire Line
+	2500 6000 2500 6075
+Text Notes 1900 5800 0    60   ~ 0
+MODE
 $EndSCHEMATC
