File: cad_files/mm5d/u2.kicad_pcb (KiCad board)
At the start: 2 copper layers, 0 parts

Commit message: 190930
Parts:
- added REF*: PIN_ARRAY_20X2, Connectors:conn2X20, F.Cu at (127.0, 99.1)
- added REF**: MountingHole_2.7mm_M2.5_Pad, Mounting_Holes:MountingHole_2.7mm_M2.5_Pad, F.Cu at (167.6, 74.9)
- added REF**: MountingHole_2.7mm_M2.5_Pad, Mounting_Holes:MountingHole_2.7mm_M2.5_Pad, F.Cu at (104.1, 74.9)
- added REF**: MountingHole_2.7mm_M2.5_Pad, Mounting_Holes:MountingHole_2.7mm_M2.5_Pad, F.Cu at (167.6, 124.5)
- added REF**: MountingHole_2.7mm_M2.5_Pad, Mounting_Holes:MountingHole_2.7mm_M2.5_Pad, F.Cu at (104.1, 124.5)
- added REF**: Pin_Header_Straight_1x20, Pin_Headers:Pin_Header_Straight_1x20, F.Cu at (118.1, 123.2)
- added REF**: Pin_Header_Straight_1x20, Pin_Headers:Pin_Header_Straight_1x20, F.Cu at (143.5, 123.2)
- added REF**: Pin_Header_Straight_1x04, Pin_Headers:Pin_Header_Straight_1x04, F.Cu at (135.9, 87.6)
Routing:
- net (no net): track 0.00 -> 414.0 mm
Other:
- board outline added: 71.1 x 57.2 mm
- net class Default: clearance 0.2 -> 0.5; trace_width 0.25 -> 0.5; via_dia 0.6 -> 2.54; via_drill 0.4 -> 0.8
- rule trace_clearance: 0.2 -> 0.5
- rule trace_min: 0.2 -> 0.5
- rule via_min_drill: 0.3 -> 0.8
- rule via_min_size: 0.4 -> 2.54
- board text added: "+3.3V"
- board text added: "+5V"
- board text added: "CE0"
- board text added: "GND"
- board text added: "GPIO12"
- board text added: "GPIO13"
- board text added: "GPIO16"
- board text added: "GPIO17"
- board text added: "GPIO18"
- board text added: "GPIO19"
- board text added: "GPIO2"
- board text added: "GPIO20"
- board text added: "GPIO21"
- board text added: "GPIO22"
- board text added: "GPIO23"
- board text added: "GPIO24"
- board text added: "GPIO25"
- board text added: "GPIO26"
- board text added: "GPIO27"
- board text added: "GPIO3"
- board text added: "GPIO4"
- board text added: "GPIO5"
- board text added: "GPIO6"
- board text added: "MOSI"
- board text added: "RXD"
- board text added: "SCLK"
- board text added: "TXD"

Commit message: 190930
Parts:
- added C201: 100u, Capacitors_THT:C_Radial_D7.5_L11.2_P2.5, F.Cu at (184.2, 118.1)
- added C202: 100n, Capacitors_THT:C_Rect_L4_W2.5_P2.5, F.Cu at (156.2, 95.2)
- added C203: 100n, Capacitors_THT:C_Rect_L4_W2.5_P2.5, F.Cu at (147.3, 100.3)
- added C204: 100n, Capacitors_THT:C_Rect_L4_W2.5_P2.5, F.Cu at (147.3, 110.5)
- added C205: 100n, Capacitors_THT:C_Rect_L4_W2.5_P2.5, F.Cu at (147.3, 102.9)
- added C206: 100n, Capacitors_THT:C_Rect_L4_W2.5_P2.5, F.Cu at (147.3, 113.0)
- added JP201: Pin_Header_Straight_2x07, Pin_Headers:Pin_Header_Straight_2x07, F.Cu at (149.9, 90.2)
- added REF**: Pin_Header_Straight_1x03, Pin_Headers:Pin_Header_Straight_1x03, F.Cu at (167.6, 102.9)
- added U201: MAX3232CPE, Housings_DIP:DIP-16_W7.62mm_LongPads, F.Cu at (153.7, 100.3)
- moved REF** 11.4 mm to (133.3, 118.1)
- moved REF** 9.16 mm to (128.3, 82.5)
- moved P201 7.18 mm to (121.9, 94.0)
- moved REF** 5.68 mm to (115.6, 118.1)
- renumbered REF* to P201
Routing:
- net (no net): track 414.0 -> 530.0 mm, vias 0 -> 6
Other:
- board size 71.1 x 57.2 mm -> 71.1 x 67.3 mm
- net class Default: via_dia 2.54 -> 2
- rule via_min_size: 2.54 -> 2
- board text added: "GND TXD RXD"
- board text added: "IO16"
- board text added: "IO20"
- board text removed: "GPIO16"
- board text removed: "GPIO20"
- board text removed: "RXD"
- board text removed: "TXD"

Commit message: 191005
Parts:
- added REF**: Pin_Header_Straight_1x01, Pin_Headers:Pin_Header_Straight_1x01, F.Cu at (147.3, 74.9)
- added REF**: Pin_Header_Straight_1x02, Pin_Headers:Pin_Header_Straight_1x02, F.Cu at (165.1, 96.5)
- added REF**: Pin_Header_Straight_2x05, Pin_Headers:Pin_Header_Straight_2x05, F.Cu at (165.1, 91.4)
- moved C201 43.1 mm to (154.9, 86.4), turned to 90 degrees
- moved REF** 10.5 mm to (165.1, 113.0), turned to 180 degrees
- moved C202 5.68 mm to (153.7, 100.3)
- moved JP201 5.68 mm to (147.3, 95.2)
- moved P201 5.68 mm to (119.4, 99.1)
- moved REF** 5.68 mm to (125.7, 87.6)
- moved C203 5.68 mm to (144.8, 105.4)
- moved C204 5.68 mm to (144.8, 115.6)
- moved C205 5.68 mm to (144.8, 108.0)
- moved C206 5.68 mm to (144.8, 118.1)
- moved REF** 5.68 mm to (113.0, 123.2)
- moved REF** 5.68 mm to (130.8, 123.2)
- moved U201 5.68 mm to (151.1, 105.4)
Routing:
- net (no net): track 530.0 -> 1117.6 mm, vias 6 -> 17
Other:
- board size 71.1 x 67.3 mm -> 71.1 x 57.2 mm
- net class Default: clearance 0.5 -> 0.2; trace_width 0.5 -> 0.25; via_dia 2 -> 0.6; via_drill 0.8 -> 0.4
- rule trace_clearance: 0.5 -> 0.2
- rule trace_min: 0.5 -> 0.2
- rule via_min_drill: 0.8 -> 0.3
- rule via_min_size: 2 -> 0.4
- board text added: "20"
- board text added: "21"
- board text added: "GPIO16"
- board text added: "NC"
- board text added: "RS232"
- board text removed: "GND TXD RXD"
- board text removed: "GPIO21"
- board text removed: "IO16"
- board text removed: "IO20"

Commit message: 191005
Parts:
- removed the REF** at (165.1, 96.5)
- added P203B: Pin_Header_Straight_2x02, Pin_Headers:Pin_Header_Straight_2x02, F.Cu at (165.1, 99.1)
- renumbered REF** to P202A, REF** to P202B, REF** to P202C, REF** to P202D, REF** to P203A, REF** to P204
Routing:
- net (no net): track 1117.6 -> 1129.6 mm, vias 17 -> 16
Other:
- board text added: "MM5D * U2 * Dn.: 59/5/7 * 2019"
- board text added: "OUT8"
- board text added: "http://www.szerafingomba.hu"
