File: cad_files/mm5d/u3.kicad_pcb (KiCad board)
At the start: 2 copper layers, 0 parts

Commit message: 191005
Parts:
- added C201: 100u, Capacitors_THT:C_Radial_D7.5_L11.2_P2.5, F.Cu at (206.4, 81.9)
- added C201: 100u, Capacitors_THT:C_Radial_D7.5_L11.2_P2.5, F.Cu at (207.6, 73.0)
- added P202C: Pin_Header_Straight_1x04, Pin_Headers:Pin_Header_Straight_1x04, F.Cu at (199.4, 77.5)
- added P202C: Pin_Header_Straight_1x04, Pin_Headers:Pin_Header_Straight_1x04, F.Cu at (195.6, 77.5)
- added P204: Pin_Header_Straight_1x03, Pin_Headers:Pin_Header_Straight_1x03, F.Cu at (191.8, 77.5)
- added REF**: MountingHole_2.7mm_M2.5_Pad, Mounting_Holes:MountingHole_2.7mm_M2.5_Pad, F.Cu at (121.9, 121.9)
- added REF**: MountingHole_2.7mm_M2.5_Pad, Mounting_Holes:MountingHole_2.7mm_M2.5_Pad, F.Cu at (161.9, 121.9)
- added REF**: MountingHole_2.7mm_M2.5_Pad, Mounting_Holes:MountingHole_2.7mm_M2.5_Pad, F.Cu at (161.9, 72.4)
- added REF**: MountingHole_2.7mm_M2.5_Pad, Mounting_Holes:MountingHole_2.7mm_M2.5_Pad, F.Cu at (121.9, 72.4)
- added REF**: Pin_Header_Straight_1x02, Pin_Headers:Pin_Header_Straight_1x02, F.Cu at (188.6, 77.5)
- added REF**: Level shifter, Connectors:levelshifter, F.Cu at (192.4, 94.0)
- added REF**: Level shifter, Connectors:levelshifter, F.Cu at (192.4, 111.8)
Other:
- board outline added: 48.3 x 57.2 mm
- board text added: "HV4 HV3 GND HV HV2 HV1"
- board text added: "LV4 LV3 GND LV LV2 LV1"
- board text added: "MM5D * U2 * Dn.: 59/5/7 * 2019"
- board text added: "http://www.szerafingomba.hu"
