File: cad_files/mm5d/u6.kicad_pcb (KiCad board)
At the start: 2 copper layers, 0 parts

Commit message: 191006
Parts:
- added D602: LED-5MM, LEDs:LED-5MM, F.Cu at (63.5, 110.5)
- added D603: LED-5MM, LEDs:LED-5MM, F.Cu at (63.5, 121.9)
- added D604: LED-5MM, LEDs:LED-5MM, F.Cu at (63.5, 133.3)
- added D605: LED-5MM, LEDs:LED-5MM, F.Cu at (63.5, 144.8)
- added P601: Pin_Header_Straight_1x13, Pin_Headers:Pin_Header_Straight_1x13, F.Cu at (77.5, 144.8)
- added R602: 330, Resistors_THT:Resistor_Horizontal_RM10mm, F.Cu at (77.5, 133.3)
- added R603: 330, Resistors_THT:Resistor_Horizontal_RM10mm, F.Cu at (80.0, 133.3)
- added R604: 330, Resistors_THT:Resistor_Horizontal_RM10mm, F.Cu at (82.5, 133.3)
- added R605: 330, Resistors_THT:Resistor_Horizontal_RM10mm, F.Cu at (85.1, 133.3)
- added R606: 270, Resistors_THT:Resistor_Horizontal_RM10mm, F.Cu at (87.6, 133.3)
- added R607: 270, Resistors_THT:Resistor_Horizontal_RM10mm, F.Cu at (90.2, 133.3)
- added R608: 270, Resistors_THT:Resistor_Horizontal_RM10mm, F.Cu at (92.7, 133.3)
- added R609: 270, Resistors_THT:Resistor_Horizontal_RM10mm, F.Cu at (95.2, 133.3)
- added R610: 270, Resistors_THT:Resistor_Horizontal_RM10mm, F.Cu at (97.8, 133.3)
- added R611: 270, Resistors_THT:Resistor_Horizontal_RM10mm, F.Cu at (100.3, 133.3)
- added R612: 270, Resistors_THT:Resistor_Horizontal_RM10mm, F.Cu at (102.9, 133.3)
- added R613: 270, Resistors_THT:Resistor_Horizontal_RM10mm, F.Cu at (105.4, 133.3)
- added R614: 270, Resistors_THT:Resistor_Horizontal_RM10mm, F.Cu at (108.0, 133.3)
- added REF**: LED-5MM, LEDs:LED-5MM, F.Cu at (193.0, 144.8)
- added REF**: LED-5MM, LEDs:LED-5MM, F.Cu at (193.0, 133.3)
- added REF**: LED-5MM, LEDs:LED-5MM, F.Cu at (193.0, 121.9)
- added REF**: LED-5MM, LEDs:LED-5MM, F.Cu at (193.0, 110.5)
- added REF**: LED-5MM, LEDs:LED-5MM, F.Cu at (128.3, 110.5)
- added REF**: MountingHole_2.7mm_M2.5, Mounting_Holes:MountingHole_2.7mm_M2.5, F.Cu at (121.9, 36.8)
- added REF**: LED-5MM, LEDs:LED-5MM, F.Cu at (128.3, 144.8)
- added REF**: MountingHole_2.7mm_M2.5, Mounting_Holes:MountingHole_2.7mm_M2.5, F.Cu at (152.4, 36.8)
- added REF**: MountingHole_2.7mm_M2.5, Mounting_Holes:MountingHole_2.7mm_M2.5, F.Cu at (143.5, 36.8)
- added REF**: MountingHole_2.7mm_M2.5, Mounting_Holes:MountingHole_2.7mm_M2.5, F.Cu at (133.3, 36.8)
- added REF**: LED-5MM, LEDs:LED-5MM, F.Cu at (63.5, 72.4)
- added REF**: LED-5MM, LEDs:LED-5MM, F.Cu at (63.5, 52.1)
- added REF**: LED-5MM, LEDs:LED-5MM, F.Cu at (128.3, 133.3)
- added REF**: LED-5MM, LEDs:LED-5MM, F.Cu at (128.3, 121.9)
Routing:
- net (no net): track 0.00 -> 1675.5 mm, vias 0 -> 16
Other:
- board outline added: 165.1 x 102.9 mm
- board text added: "Display module"
- board text added: "LED1"
- board text added: "LED10"
- board text added: "LED11"
- board text added: "LED12"
- board text added: "LED13"
- board text added: "LED2"
- board text added: "LED3"
- board text added: "LED4"
- board text added: "LED5"
- board text added: "LED6"
- board text added: "LED7"
- board text added: "LED8"
- board text added: "LED9"
