File: cad_files/mm5d/u4.sch (KiCad schematic (older format))
At the start: 33 parts, among them P602 CONN_01X05, SW601 SWITCH_1P

Commit message: 200128
Parts:
- removed C601, C602: 4.7u, symbol CP
- removed P602: CONN_01X05, symbol CONN_01X05
- renumbered D601 to D401, D602 to D402, D603 to D403, D604 to D404, D605 to D405, D606 to D406, D607 to D407, D608 to D408, D609 to D409, D610 to D410, D611 to D411, D612 to D412, D613 to D413, D614 to D414, R601 to R401, R602 to R402, R603 to R403, R604 to R404, R605 to R405, R606 to R406, R607 to R407, R608 to R408, R609 to R409, R610 to R410, R611 to R411, R612 to R412, R613 to R413, R614 to R414, R615 to R415, SW601 to SW401
Connections:
- net labels added: VCC3, VCC5
- net labels removed: CE0, MOSI, SCLK
- wire segments 78 -> 70
Other:
- note removed: "connector of 32x8 matrix display modul"
- moved on the sheet: D401, D402, D403, D404, D405, D406, D407, D408, D409, D410, D411, D412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

Commit message: 200129
Other:
- moved on the sheet: D401, D402, D403, D404, D405, D406, D407, D408, D409, D410, D411, D412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

Commit message: 200130
Connections:
- net +5V is gone; now on net VCC3: D401.2 (A), D402.2 (A), D403.2 (A), D404.2 (A), D405.2 (A)
- net +3V3 renamed VCC3
- net VCC3: now also R415.1; no longer R415.2
- net SW-MODE renamed SW
- net SW: now also R415.2; no longer R415.1
Other:
- moved on the sheet: D401, D402, D403, D404, D405, D406, D407, D408, D409, D410, D411, D412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

Commit message: 200213
Parts:
- R415: value 1k -> 4.7k
Changed lines of the file:
@@
 P 3025 5000
 F 0 "R415" V 3125 5000 50  0000 C CNN
-F 1 "1k" V 2900 5000 50  0000 C CNN
+F 1 "4.7k" V 2900 5000 50  0000 C CNN
 F 2 "" V 2955 5000 50  0000 C CNN
 F 3 "" H 3025 5000 50  0000 C CNN
