File: cad_files/mm5d/u5.sch (KiCad schematic (older format))
At the start: 17 parts, among them U301 Level_shifter_4, U302 Level_shifter_4

Commit message: 200129
Parts:
- R509: renamed from R?; value 100 -> 4,7k
- gave numbers to parts that had none: 2
- renumbered D301 to D501, D302 to D502, D303 to D503, D304 to D504, R301 to R501, R302 to R502, R303 to R503, R304 to R504, R305 to R505, R306 to R506, R307 to R507, R308 to R508, U302 to U501, U301 to U502
Connections:
- net +3.3V is gone; now on net VCC5: U501.~ (LV4), U502.~ (LV4)
- net +5V is gone; now on net VCC5: J502.1, R505.1, R506.1, R507.1, R508.1, R509.1, U501.~ (LV4), U502.~ (LV4)
- net VCC5: now reaches U502.~ (LV4)
- new net VCC3: U501.~ (LV4), U502.~ (LV4)
Other:
- note added: "level shifter"
Changed lines of the file:
@@
 Rev "200128"
 Comp "Pozsar Zsolt -  http://www.szerafingomba.hu"
-Comment1 "Unit U3"
-Comment2 "Input module"
+Comment1 "Module U5"
+Comment2 "Inputs"
 Comment3 ""
 Comment4 "Draw no.: 59/2/4"
@@
 OUT4
 Text HLabel 8775 2150 2    60   Input ~ 0
-+5V
+VCC5
 Text HLabel 8775 5175 2    60   UnSpc ~ 0
 GND
 Text HLabel 8775 2250 2    60   Input ~ 0
-+3.3V
+VCC3
 Text HLabel 8775 4975 2    60   BiDi ~ 0
 SENSOR
 $Comp
-L R R305
+L R R505
 U 1 1 5D8801CC
 P 3300 2400
-F 0 "R305" V 3175 2300 50  0000 C CNN
+F 0 "R505" V 3175 2300 50  0000 C CNN
 F 1 "1k" V 3400 2475 50  0000 C CNN
 F 2 "" V 3230 2400 50  0000 C CNN
@@
 $EndComp
 $Comp
-L D D301
+L D D501
 U 1 1 5D880243
 P 3300 3850
-F 0 "D301" H 3300 3975 50  0000 C CNN
+F 0 "D501" H 3300 3975 50  0000 C CNN
 F 1 "1N4001" V 3775 3875 50  0000 C CNN
 F 2 "" H 3300 3850 50  0000 C CNN
@@
 $EndComp
 $Comp
-L R R306
+L R R506
 U 1 1 5D880D19
 P 3600 2400
-F 0 "R306" V 3475 2300 50  0000 C CNN
+F 0 "R506" V 3475 2300 50  0000 C CNN
 F 1 "1k" V 3700 2475 50  0000 C CNN
 F 2 "" V 3530 2400 50  0000 C CNN
@@
 $EndComp
 $Comp
-L R R307
+L R R507
 U 1 1 5D880E74
 P 3900 2400
-F 0 "R307" V 3775 2300 50  0000 C CNN
+F 0 "R507" V 3775 2300 50  0000 C CNN
 F 1 "1k" V 4000 2475 50  0000 C CNN
 F 2 "" V 3830 2400 50  0000 C CNN
@@
 $EndComp
 $Comp
-L R R308
+L R R508
 U 1 1 5D880E7B
 P 4200 2400
-F 0 "R308" V 4075 2300 50  0000 C CNN
+F 0 "R508" V 4075 2300 50  0000 C CNN
 F 1 "1k" V 4300 2475 50  0000 C CNN
 F 2 "" V 4130 2400 50  0000 C CNN
@@
 $EndComp
 $Comp
-L D D302
+L D D502
 U 1 1 5D880E90
 P 3600 3850
-F 0 "D302" H 3600 3975 50  0000 C CNN
+F 0 "D502" H 3600 3975 50  0000 C CNN
 F 1 "1N4001" V 3975 3850 50  0000 C CNN
 F 2 "" H 3600 3850 50  0000 C CNN
@@
 $EndComp
 $Comp
-L D D303
+L D D503
 U 1 1 5D880ED6
 P 3900 3850
-F 0 "D303" H 3900 3975 50  0000 C CNN
+F 0 "D503" H 3900 3975 50  0000 C CNN
 F 1 "1N4001" V 4375 3850 50  0000 C CNN
 F 2 "" H 3900 3850 50  0000 C CNN
@@
 $EndComp
 $Comp
-L D D304
+L D D504
 U 1 1 5D880F1D
 P 4200 3850
-F 0 "D304" H 4200 3975 50  0000 C CNN
+F 0 "D504" H 4200 3975 50  0000 C CNN
 F 1 "1N4001" V 4575 3850 50  0000 C CNN
 F 2 "" H 4200 3850 50  0000 C CNN
@@
 $EndComp
 $Comp
-L R R301
+L R R501
 U 1 1 5D881151
 P 2925 2850
-F 0 "R301" V 2850 2625 50  0000 C CNN
+F 0 "R501" V 2850 2625 50  0000 C CNN
 F 1 "100" V 3000 3050 50  0000 C CNN
 F 2 "" V 2855 2850 50  0000 C CNN
@@
 $EndComp
 $Comp
-L R R302
+L R R502
 U 1 1 5D8811B2
 P 2925 3050
-F 0 "R302" V 2850 2825 50  0000 C CNN
+F 0 "R502" V 2850 2825 50  0000 C CNN
 F 1 "100" V 3000 3250 50  0000 C CNN
 F 2 "" V 2855 3050 50  0000 C CNN
@@
 $EndComp
 $Comp
-L R R303
+L R R503
 U 1 1 5D8811EE
 P 2925 3250
-F 0 "R303" V 2850 3025 50  0000 C CNN
+F 0 "R503" V 2850 3025 50  0000 C CNN
 F 1 "100" V 3000 3450 50  0000 C CNN
 F 2 "" V 2855 3250 50  0000 C CNN
@@
 $EndComp
 $Comp
-L R R304
+L R R504
 U 1 1 5D881235
 P 2925 3450
-F 0 "R304" V 2850 3225 50  0000 C CNN
+F 0 "R504" V 2850 3225 50  0000 C CNN
 F 1 "100" V 3000 3650 50  0000 C CNN
 F 2 "" V 2855 3450 50  0000 C CNN
@@
 $EndComp
 $Comp
-L Level_shifter_4 U302
+L Level_shifter_4 U501
 U 1 1 5D873257
 P 6850 3000
-F 0 "U302" V 6525 3525 60  0000 C CNN
+F 0 "U501" H 6600 3425 60  0000 C CNN
 F 1 "Level_shifter_4" H 6850 2550 60  0001 C CNN
 F 2 "" H 6850 2700 60  0000 C CNN
@@
 $EndComp
 $Comp
-L Level_shifter_4 U301
+L Level_shifter_4 U502
 U 1 1 5D875485
 P 6850 4925
-F 0 "U301" V 6525 5425 60  0000 C CNN
+F 0 "U502" H 6600 5350 60  0000 C CNN
 F 1 "Level_shifter_4" H 6850 4475 60  0001 C CNN
 F 2 "" H 6850 4625 60  0000 C CNN
@@
 $EndComp
 $Comp
-L Screw_Terminal_1x05 J?
+L Screw_Terminal_1x05 J501
 U 1 1 5E3206E7
 P 2275 3250
-F 0 "J?" H 2275 3800 50  0000 C TNN
-F 1 "Screw_Terminal_1x05" V 2125 3250 50  0000 C TNN
+F 0 "J501" H 2300 3875 50  0000 C TNN
+F 1 "Screw_Terminal_1x05" V 2125 3250 50  0001 C TNN
 F 2 "" H 2275 2725 50  0001 C CNN
 F 3 "" H 2250 3550 50  0001 C CNN
@@
 $EndComp
 $Comp
-L Screw_Terminal_1x03 J?
+L Screw_Terminal_1x03 J502
 U 1 1 5E320756
 P 2275 4975
-F 0 "J?" H 2275 5325 50  0000 C TNN
-F 1 "Screw_Terminal_1x03" V 2125 4975 50  0000 C TNN
+F 0 "J502" H 2300 5375 50  0000 C TNN
+F 1 "Screw_Terminal_1x03" V 2125 4975 50  0001 C TNN
 F 2 "" H 2275 4650 50  0001 C CNN
 F 3 "" H 2250 5075 50  0001 C CNN
@@
 	1    0    0    -1
 $EndComp
+$Comp
+L R R509
+U 1 1 5E321F52
+P 2925 4875
+F 0 "R509" V 2750 4875 50  0000 C CNN
+F 1 "4,7k" V 3100 4875 50  0000 C CNN
+F 2 "" V 2855 4875 50  0000 C CNN
+F 3 "" H 2925 4875 50  0000 C CNN
+	1    2925 4875
+	0    1    1    0
+$EndComp
+NoConn ~ 7500 5075
+NoConn ~ 7500 4875
+NoConn ~ 7500 4775
+Text Notes 6575 3450 0    60   ~ 0
+level shifter
+Text Notes 6575 5375 0    60   ~ 0
+level shifter
+Text Label 8700 2150 2    60   ~ 0
++5V
+Text Label 8700 2250 2    60   ~ 0
++3.3V
 Wire Wire Line
 	3075 2850 6200 2850
@@
 Wire Wire Line
 	5950 4675 6200 4675
-$Comp
-L R R?
-U 1 1 5E321F52
-P 2925 4875
-F 0 "R?" V 2850 4650 50  0000 C CNN
-F 1 "100" V 3000 5075 50  0000 C CNN
-F 2 "" V 2855 4875 50  0000 C CNN
-F 3 "" H 2925 4875 50  0000 C CNN
-	1    2925 4875
-	0    1    1    0
-$EndComp
 Wire Wire Line
 	2775 4875 2700 4875
@@
 	7850 3250 7850 5175
 Connection ~ 7850 5175
-NoConn ~ 7500 5075
-NoConn ~ 7500 4875
-NoConn ~ 7500 4775
 Wire Wire Line
 	6200 4775 6100 4775

Commit message: 200213
Parts:
- R505, R506, R507, R508: value 1k -> 4.7k
- R509: value 4,7k -> 4.7k
Changed lines of the file:
@@
 P 3300 2400
 F 0 "R505" V 3175 2300 50  0000 C CNN
-F 1 "1k" V 3400 2475 50  0000 C CNN
+F 1 "4.7k" V 3400 2475 50  0000 C CNN
 F 2 "" V 3230 2400 50  0000 C CNN
 F 3 "" H 3300 2400 50  0000 C CNN
@@
 P 3600 2400
 F 0 "R506" V 3475 2300 50  0000 C CNN
-F 1 "1k" V 3700 2475 50  0000 C CNN
+F 1 "4.7k" V 3700 2475 50  0000 C CNN
 F 2 "" V 3530 2400 50  0000 C CNN
 F 3 "" H 3600 2400 50  0000 C CNN
@@
 P 3900 2400
 F 0 "R507" V 3775 2300 50  0000 C CNN
-F 1 "1k" V 4000 2475 50  0000 C CNN
+F 1 "4.7k" V 4000 2475 50  0000 C CNN
 F 2 "" V 3830 2400 50  0000 C CNN
 F 3 "" H 3900 2400 50  0000 C CNN
@@
 P 4200 2400
 F 0 "R508" V 4075 2300 50  0000 C CNN
-F 1 "1k" V 4300 2475 50  0000 C CNN
+F 1 "4.7k" V 4300 2475 50  0000 C CNN
 F 2 "" V 4130 2400 50  0000 C CNN
 F 3 "" H 4200 2400 50  0000 C CNN
@@
 P 2925 4875
 F 0 "R509" V 2750 4875 50  0000 C CNN
-F 1 "4,7k" V 3100 4875 50  0000 C CNN
+F 1 "4.7k" V 3100 4875 50  0000 C CNN
 F 2 "" V 2855 4875 50  0000 C CNN
 F 3 "" H 2925 4875 50  0000 C CNN
