File: cad_files/mm5d-u5-pcb/u5.kicad_pcb (KiCad board)
At the start: 2 copper layers, 71.1 x 57.2 mm, 20 parts, among them P201 PIN_ARRAY_20X2, P202A Pin_Header_Straight_1x20, P202B Pin_Header_Straight_1x20, P202C Pin_Header_Straight_1x04, P202D Pin_Header_Straight_1x01, P203A Pin_Header_Straight_2x05, P203B Pin_Header_Straight_2x02, P204 Pin_Header_Straight_1x03, U201 MAX3232CPE

Commit message: 200219
Parts:
- removed C201: 100u, Capacitors_THT:C_Radial_D7.5_L11.2_P2.5
- removed C202, C203, C204, C205, C206: 100n, Capacitors_THT:C_Rect_L4_W2.5_P2.5
- removed JP201: Pin_Header_Straight_2x07, Pin_Headers:Pin_Header_Straight_2x07
- removed P201: PIN_ARRAY_20X2, Connectors:conn2X20
- removed P202A, P202B: Pin_Header_Straight_1x20, Pin_Headers:Pin_Header_Straight_1x20
- removed P202C: Pin_Header_Straight_1x04, Pin_Headers:Pin_Header_Straight_1x04
- removed P202D: Pin_Header_Straight_1x01, Pin_Headers:Pin_Header_Straight_1x01
- removed P203A: Pin_Header_Straight_2x05, Pin_Headers:Pin_Header_Straight_2x05
- removed P203B: Pin_Header_Straight_2x02, Pin_Headers:Pin_Header_Straight_2x02
- removed P204: Pin_Header_Straight_1x03, Pin_Headers:Pin_Header_Straight_1x03
- removed U201: MAX3232CPE, Housings_DIP:DIP-16_W7.62mm_LongPads
- added D501: D4, Discret:D4, F.Cu at (149.9, 108.0)
- added D502: D4, Discret:D4, F.Cu at (149.9, 100.3)
- added D503: D4, Discret:D4, F.Cu at (149.9, 92.7)
- added D504: D4, Discret:D4, F.Cu at (149.9, 85.1)
- added J501: SolderWirePad_single_1mmDrill, Wire_Pads:SolderWirePad_single_1mmDrill, F.Cu at (161.3, 108.0)
- added J502: SolderWirePad_single_1mmDrill, Wire_Pads:SolderWirePad_single_1mmDrill, F.Cu at (161.3, 118.1)
- added J502: SolderWirePad_single_1mmDrill, Wire_Pads:SolderWirePad_single_1mmDrill, F.Cu at (161.3, 113.0)
- added R501: R4, Discret:R4, F.Cu at (149.9, 104.1)
- added R502: R4, Discret:R4, F.Cu at (149.9, 96.5)
- added R503: R4, Discret:R4, F.Cu at (149.9, 88.9)
- added R504: R4, Discret:R4, F.Cu at (149.9, 81.3)
- added R505: R4, Discret:R4, F.Cu at (139.7, 104.1)
- added R506: R4, Discret:R4, F.Cu at (135.9, 101.6)
- added R507: R4, Discret:R4, F.Cu at (139.7, 83.8)
- added R508: R4, Discret:R4, F.Cu at (135.9, 81.3)
- added R509: R4, Discret:R4, F.Cu at (149.9, 111.8)
- added REF**: SolderWirePad_single_1mmDrill, Wire_Pads:SolderWirePad_single_1mmDrill, F.Cu at (161.3, 101.6)
- added REF**: SolderWirePad_single_1mmDrill, Wire_Pads:SolderWirePad_single_1mmDrill, F.Cu at (161.3, 81.3)
- added REF**: SolderWirePad_single_0-8mmDrill, Wire_Pads:SolderWirePad_single_0-8mmDrill, F.Cu at (132.1, 106.7)
- added REF**: SolderWirePad_single_0-8mmDrill, Wire_Pads:SolderWirePad_single_0-8mmDrill, F.Cu at (132.1, 114.3)
- added REF**: SolderWirePad_single_1mmDrill, Wire_Pads:SolderWirePad_single_1mmDrill, F.Cu at (161.3, 91.4)
- added REF**: SolderWirePad_single_1mmDrill, Wire_Pads:SolderWirePad_single_1mmDrill, F.Cu at (161.3, 96.5)
- added REF**: SolderWirePad_single_1mmDrill, Wire_Pads:SolderWirePad_single_1mmDrill, F.Cu at (161.3, 86.4)
- added REF**: Socket_Strip_Straight_1x08, Socket_Strips:Socket_Strip_Straight_1x08, F.Cu at (109.2, 90.2)
- added U501: Level shifter, Connectors:levelshifter, F.Cu at (116.8, 86.4)
- added U502: Level shifter, Connectors:levelshifter, F.Cu at (116.8, 109.2)
- moved REF** 1.27 mm to (105.4, 124.5)
- moved REF** 1.27 mm to (105.4, 74.9)
- moved REF** 1.27 mm to (166.4, 74.9)
- moved REF** 1.27 mm to (166.4, 124.5)
Routing:
- net (no net): track 1129.6 -> 638.2 mm, vias 16 -> 0
Other:
- board text added: "2019"
- board text added: "Data"
- board text added: "Dn.: 59/5/8"
- board text added: "In1"
- board text added: "In2"
- board text added: "In3"
- board text added: "In4"
- board text added: "MM5D/U5"
- board text added: "OUT1"
- board text added: "OUT2"
- board text added: "OUT3"
- board text added: "OUT4"
- board text added: "SENS"
- board text added: "VCC3"
- board text added: "VCC5"
- board text removed: "+3.3V"
- board text removed: "20"
- board text removed: "21"
- board text removed: "CE0"
- board text removed: "GPIO12"
- board text removed: "GPIO13"
- board text removed: "GPIO16"
- board text removed: "GPIO17"
- board text removed: "GPIO18"
- board text removed: "GPIO19"
- board text removed: "GPIO2"
- board text removed: "GPIO22"
- board text removed: "GPIO23"
- board text removed: "GPIO24"
- board text removed: "GPIO25"
- board text removed: "GPIO26"
- board text removed: "GPIO27"
- board text removed: "GPIO3"
- board text removed: "GPIO4"
- board text removed: "GPIO5"
- board text removed: "GPIO6"
- board text removed: "MM5D * U2 * Dn.: 59/5/7 * 2019"
- board text removed: "MOSI"
- board text removed: "NC"
- board text removed: "OUT8"
- board text removed: "RS232"
- board text removed: "SCLK"
- board text removed: "http://www.szerafingomba.hu"
