File: cad_files/mm5d-u4-pcb/u4.kicad_pcb (KiCad board)
At the start: 2 copper layers, 48.3 x 57.2 mm, 12 parts, among them P202C Pin_Header_Straight_1x04, P204 Pin_Header_Straight_1x03

Commit message: 200215
Parts:
- removed C201 (x2): 100u, Capacitors_THT:C_Radial_D7.5_L11.2_P2.5
- removed P202C (x2): Pin_Header_Straight_1x04, Pin_Headers:Pin_Header_Straight_1x04
- removed P204: Pin_Header_Straight_1x03, Pin_Headers:Pin_Header_Straight_1x03
- removed the REF** at (121.9, 121.9)
- removed the REF** at (161.9, 121.9)
- removed the REF** at (188.6, 77.5)
- removed the REF** at (192.4, 94.0)
- removed the REF** at (192.4, 111.8)
- added D401: Pin_Header_Straight_2x01, Pin_Headers:Pin_Header_Straight_2x01, F.Cu at (119.4, 83.8)
- added D402: Pin_Header_Straight_2x01, Pin_Headers:Pin_Header_Straight_2x01, F.Cu at (123.2, 83.8)
- added D403: Pin_Header_Straight_2x01, Pin_Headers:Pin_Header_Straight_2x01, F.Cu at (127.0, 83.8)
- added D404: Pin_Header_Straight_2x01, Pin_Headers:Pin_Header_Straight_2x01, F.Cu at (130.8, 83.8)
- added D405: Pin_Header_Straight_2x01, Pin_Headers:Pin_Header_Straight_2x01, F.Cu at (134.6, 83.8)
- added D406: Pin_Header_Straight_2x01, Pin_Headers:Pin_Header_Straight_2x01, F.Cu at (138.4, 83.8)
- added D407: Pin_Header_Straight_2x01, Pin_Headers:Pin_Header_Straight_2x01, F.Cu at (142.2, 83.8)
- added D408: Pin_Header_Straight_2x01, Pin_Headers:Pin_Header_Straight_2x01, F.Cu at (146.1, 83.8)
- added D409: Pin_Header_Straight_2x01, Pin_Headers:Pin_Header_Straight_2x01, F.Cu at (149.9, 83.8)
- added D410: Pin_Header_Straight_2x01, Pin_Headers:Pin_Header_Straight_2x01, F.Cu at (153.7, 83.8)
- added D411: Pin_Header_Straight_2x01, Pin_Headers:Pin_Header_Straight_2x01, F.Cu at (157.5, 83.8)
- added D412: Pin_Header_Straight_2x01, Pin_Headers:Pin_Header_Straight_2x01, F.Cu at (161.3, 83.8)
- added D413: Pin_Header_Straight_2x01, Pin_Headers:Pin_Header_Straight_2x01, F.Cu at (165.1, 83.8)
- added D414: Pin_Header_Straight_2x01, Pin_Headers:Pin_Header_Straight_2x01, F.Cu at (168.9, 81.3)
- added R401: R4, Discret:R4, F.Cu at (119.4, 94.0)
- added R402: R4, Discret:R4, F.Cu at (123.2, 94.0)
- added R403: R4, Discret:R4, F.Cu at (127.0, 94.0)
- added R404: R4, Discret:R4, F.Cu at (130.8, 94.0)
- added R405: R4, Discret:R4, F.Cu at (134.6, 94.0)
- added R406: R4, Discret:R4, F.Cu at (138.4, 94.0)
- added R407: R4, Discret:R4, F.Cu at (142.2, 94.0)
- added R408: R4, Discret:R4, F.Cu at (146.1, 94.0)
- added R409: R4, Discret:R4, F.Cu at (149.9, 94.0)
- added R410: R4, Discret:R4, F.Cu at (153.7, 94.0)
- added R411: R4, Discret:R4, F.Cu at (157.5, 94.0)
- added R412: R4, Discret:R4, F.Cu at (161.3, 94.0)
- added R413: R4, Discret:R4, F.Cu at (165.1, 94.0)
- added R414: R4, Discret:R4, F.Cu at (168.9, 94.0)
- added R415: R4, Discret:R4, F.Cu at (172.7, 94.0)
- added REF**: Pin_Header_Straight_1x16, Pin_Headers:Pin_Header_Straight_1x16, F.Cu at (129.5, 108.0)
- added REF**: SolderWirePad_single_0-8mmDrill, Wire_Pads:SolderWirePad_single_0-8mmDrill, F.Cu at (177.8, 99.1)
- added REF**: SolderWirePad_single_0-8mmDrill, Wire_Pads:SolderWirePad_single_0-8mmDrill, F.Cu at (177.8, 88.9)
- added SW401: Pin_Header_Straight_2x01, Pin_Headers:Pin_Header_Straight_2x01, F.Cu at (172.7, 83.8)
- moved REF** 67.5 mm to (185.4, 95.2)
- moved REF** 58.6 mm to (108.0, 95.2)
Routing:
- net (no net): track 0.00 -> 512.4 mm
Other:
- board size 48.3 x 57.2 mm -> 87.6 x 40.6 mm
- board text added: "2019"
- board text added: "Dn.: 59/5/7"
- board text added: "GND"
- board text added: "LED1"
- board text added: "LED10"
- board text added: "LED11"
- board text added: "LED12"
- board text added: "LED13"
- board text added: "LED2"
- board text added: "LED3"
- board text added: "LED4"
- board text added: "LED5"
- board text added: "LED6"
- board text added: "LED7"
- board text added: "LED8"
- board text added: "LED9"
- board text added: "MM5D/U5"
- board text added: "SW"
- board text added: "VCC3"
- board text removed: "HV4 HV3 GND HV HV2 HV1"
- board text removed: "LV4 LV3 GND LV LV2 LV1"
- board text removed: "MM5D * U2 * Dn.: 59/5/7 * 2019"
- board text removed: "http://www.szerafingomba.hu"
