File: cad_files/mm5d-pcb/mm5d.kicad_pcb (KiCad board)
At the start: 2 copper layers, 48.3 x 57.2 mm, 24 parts, among them J1 SolderWirePad_single_1mmDrill, T1 TO39EBC

Commit message: 200224
Routing:
- net (no net): track 393.2 -> 398.3 mm
Changed lines of the file:
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@@
-(kicad_pcb (version 4) (host pcbnew 4.0.7)
+(kicad_pcb (version 4) (host pcbnew 4.0.5+dfsg1-4)
   (general
     (links 0)
     (no_connects 0)
-    (area 118.034999 68.504999 166.445001 125.805001)
+    (area 109.862857 65.015713 178.029999 132.240001)
     (thickness 1.6)
     (drawings 33)
-    (tracks 74)
+    (tracks 75)
     (zones 0)
     (modules 24)
@@
     (visible_elements 7FFEEF7F)
     (pcbplotparams
-      (layerselection 0x01060_80000000)
+      (layerselection 0x00000_80000000)
       (usegerberextensions false)
       (excludeedgelayer false)
       (linewidth 0.150000)
-      (plotframeref false)
+      (plotframeref true)
       (viasonmask false)
       (mode 1)
@@
       (padsonsilk false)
       (subtractmaskfromsilk false)
-      (outputformat 1)
-      (mirror false)
-      (drillshape 0)
+      (outputformat 5)
+      (mirror true)
+      (drillshape 1)
       (scaleselection 1)
       (outputdirectory ""))
@@
   (gr_line (start 165.1 125.73) (end 166.37 125.73) (angle 90) (layer Edge.Cuts) (width 0.15))
   (gr_line (start 158.115 125.73) (end 165.1 125.73) (angle 90) (layer Edge.Cuts) (width 0.15))
+  (segment (start 134.62 119.38) (end 139.7 119.38) (width 2.5) (layer B.Cu) (net 0))
   (segment (start 133.35 102.87) (end 133.35 112.395) (width 2.5) (layer B.Cu) (net 0))
   (segment (start 133.35 102.87) (end 121.92 102.87) (width 2.5) (layer B.Cu) (net 0))
