File: cad_files/mm5d-sch/mm5d.sch (KiCad schematic (older format))
At the start: 22 parts, among them J1 Screw_Terminal_1x03, J2 DB9 female, J3 CONN_02X20, J4 CONN_02X20, J5 CONN_02X20, SW1 SWITCH_1P, T1 2N2219, U3 Matrix_display, U6 Relay_panel, U7 Relay_panel

Commit message: 200223
Parts:
- renumbered J4 to JP1, J3 to JP2, J5 to JP4
Connections:
- no-connect marks 81 -> 80
Other:
- note added: "All unit connected to Raspberry Pi via 3 slot GPIO expansion card\n by JP1, JP2 and JP4 plugs."
- note removed: "All unit connected to Raspberry Pi via 3 slot GPIO expansion module by J3-5 plugs."
- moved on the sheet: U7
Changed lines of the file:
@@
 L Relay_panel U7
 U 1 1 5D85EA39
-P 8650 1350
-F 0 "U7" V 9050 1850 60  0000 C CNN
-F 1 "Relay_panel" H 8650 600 60  0001 C CNN
-F 2 "" H 8650 1350 60  0000 C CNN
-F 3 "" H 8650 1350 60  0000 C CNN
-	1    8650 1350
+P 8650 1250
+F 0 "U7" V 9050 1750 60  0000 C CNN
+F 1 "Relay_panel" H 8650 500 60  0001 C CNN
+F 2 "" H 8650 1250 60  0000 C CNN
+F 3 "" H 8650 1250 60  0000 C CNN
+	1    8650 1250
 	0    -1   -1   0
 $EndComp
@@
 $EndComp
 $Comp
-L CONN_02X20 J4
+L CONN_02X20 JP1
 U 1 1 5E3076A1
 P 5750 3500
-F 0 "J4" H 5750 4550 50  0000 C CNN
+F 0 "JP1" H 5750 4550 50  0000 C CNN
 F 1 "CONN_02X20" V 5750 3500 50  0001 C CNN
 F 2 "" H 5750 2550 50  0000 C CNN
@@
 $EndComp
 $Comp
-L CONN_02X20 J3
+L CONN_02X20 JP2
 U 1 1 5E3088F3
 P 2300 3500
-F 0 "J3" H 2300 4550 50  0000 C CNN
+F 0 "JP2" H 2300 4550 50  0000 C CNN
 F 1 "CONN_02X20" V 2300 3500 50  0001 C CNN
 F 2 "" H 2300 2550 50  0000 C CNN
@@
 $EndComp
 $Comp
-L CONN_02X20 J5
+L CONN_02X20 JP4
 U 1 1 5E3094F6
 P 9650 3500
-F 0 "J5" H 9650 4550 50  0000 C CNN
+F 0 "JP4" H 9650 4550 50  0000 C CNN
 F 1 "CONN_02X20" V 9650 3500 50  0001 C CNN
 F 2 "" H 9650 2550 50  0000 C CNN
@@
 Text Label 8200 4750 0    60   ~ 0
 +5V
-Text Label 8200 2300 0    60   ~ 0
+Text Label 9150 2300 0    60   ~ 0
 +5V
 Text Label 9950 2750 0    60   ~ 0
@@
 Text Label 9350 2850 2    60   ~ 0
 GPIO04
-NoConn ~ 8900 2000
+NoConn ~ 8900 1900
 Text Label 2000 4350 2    60   ~ 0
 GPIO26
@@
 	8200 4750 10300 4750
 Wire Wire Line
-	10300 2650 10300 5300
+	10300 4750 10300 2650
 Wire Wire Line
 	10300 2650 9900 2650
@@
 	9400 2650 8600 2650
 Wire Wire Line
-	8600 2650 8600 2000
-Wire Wire Line
-	8700 2000 8700 2750
+	8600 2650 8600 1900
+Wire Wire Line
+	8700 1900 8700 2750
 Wire Wire Line
 	8700 2750 9400 2750
 Wire Wire Line
-	8800 2000 8800 2850
+	8800 1900 8800 2850
 Wire Wire Line
 	8800 2850 9400 2850
 Wire Wire Line
-	8200 2000 8200 2300
+	8200 1900 8200 2300
 Wire Wire Line
 	8200 2300 10300 2300
@@
 	10400 2200 9100 2200
 Wire Wire Line
-	9100 2200 9100 2000
+	9100 2200 9100 1900
 Wire Wire Line
 	6300 5750 6300 6300
@@
 Wire Wire Line
 	4425 6600 4425 6750
-Text Notes 7150 6300 0    60   ~ 0
-All unit connected to Raspberry Pi via 3 slot GPIO expansion module by J3-5 plugs.
+Text Notes 7975 6350 0    60   ~ 0
+All unit connected to Raspberry Pi via 3 slot GPIO expansion card\n                   by JP1, JP2 and JP4 plugs.
 $Comp
 L R R1
@@
 $EndComp
 Wire Wire Line
-	10300 5300 10250 5300
-Connection ~ 10300 4750
+	10250 5300 10600 5300
 Wire Wire Line
 	8400 4925 8400 4850
@@
 Connection ~ 9300 4850
 Wire Wire Line
-	8400 2100 8400 2000
+	8400 2100 8400 1900
 Text Notes 9500 5550 0    60   ~ 0
 Disable outputs\n  (key switch)
 NoConn ~ 8300 4925
-NoConn ~ 8300 2000
 Text Label 9150 2100 0    60   ~ 0
 +5V-Relay
 Text Label 9550 4850 0    60   ~ 0
 +5V-Relay
-Text Label 10300 5250 1    60   ~ 0
+Text Label 10450 5300 2    60   ~ 0
 +5V
 Text Label 7900 2200 1    60   ~ 0
@@
 Connection ~ 3900 6600
 Connection ~ 4100 6600
+Wire Wire Line
+	8300 1900 8300 2000
+Wire Wire Line
+	8300 2000 10600 2000
+Wire Wire Line
+	10600 2000 10600 5300
+Text Label 9325 2000 2    60   ~ 0
++5V
+Text Label 7550 3650 3    60   ~ 0
+GND
 $EndSCHEMATC

Commit message: 200418
Connections:
- net +5V: no longer J2.9 (P9), JP1.4 (P4), JP2.2 (P2), JP2.4 (P4), JP4.2 (P2), JP4.4 (P4)
- no-connect marks 80 -> 85
Other:
- moved on the sheet: C4
Changed lines of the file:
@@
 Text Label 6050 2550 0    60   ~ 0
 +5V
-Text Label 9950 2550 0    60   ~ 0
-+5V
-Text Label 9950 2650 0    60   ~ 0
-+5V
-Text Label 8200 4750 0    60   ~ 0
-+5V
-Text Label 9150 2300 0    60   ~ 0
+Text Label 8200 4925 1    60   ~ 0
 +5V
 Text Label 9950 2750 0    60   ~ 0
@@
 	4400 3350 5500 3350
 Wire Wire Line
-	6000 2550 6325 2550
-Wire Wire Line
-	6325 2550 6325 1950
-Wire Wire Line
-	6325 1950 3300 1950
-Wire Wire Line
-	3300 1950 3300 1150
+	6450 2550 6000 2550
+Wire Wire Line
+	3300 1150 3300 2350
 Wire Wire Line
 	3300 1150 4000 1150
@@
 	9100 4650 9100 4925
 Wire Wire Line
-	8200 4925 8200 4750
-Wire Wire Line
-	8200 4750 10300 4750
-Wire Wire Line
-	10300 4750 10300 2650
-Wire Wire Line
-	10300 2650 9900 2650
-Wire Wire Line
 	9400 2650 8600 2650
 Wire Wire Line
@@
 Wire Wire Line
 	8800 2850 9400 2850
-Wire Wire Line
-	8200 1900 8200 2300
-Wire Wire Line
-	8200 2300 10300 2300
-Wire Wire Line
-	10300 2300 10300 2550
-Wire Wire Line
-	10300 2550 9900 2550
 Wire Wire Line
 	9900 3150 10400 3150
@@
 	2450 5250 2450 6300
 Wire Wire Line
-	2550 2650 3200 2650
-Wire Wire Line
-	3200 2650 3200 5350
+	3200 3050 3200 5350
 Wire Wire Line
 	3200 5350 2050 5350
@@
 Wire Wire Line
 	3700 6700 3700 6650
-Text Label 2600 2550 0    60   ~ 0
-+5V
-Wire Wire Line
-	3900 2950 3900 6700
+Wire Wire Line
+	3900 2950 3900 3850
+Wire Wire Line
+	3900 3850 3900 4550
+Wire Wire Line
+	3900 4550 3900 5650
+Wire Wire Line
+	3900 5650 3900 6600
+Wire Wire Line
+	3900 6600 3900 6700
 Wire Wire Line
 	3500 6100 3500 6200
@@
 	3500 6200 3700 6200
 Wire Wire Line
-	3450 4400 4150 4400
+	3450 4400 3700 4400
+Wire Wire Line
+	3700 4400 4150 4400
 Connection ~ 3700 6200
 Wire Wire Line
@@
 	3500 5650 3900 5650
 Wire Wire Line
-	3450 3850 4150 3850
+	3450 3850 3900 3850
+Wire Wire Line
+	3900 3850 4150 3850
 Connection ~ 3900 5650
 Text Notes 3575 7275 0    60   ~ 0
   Power in\n(5V 2.5A DC)
 Wire Wire Line
-	1750 1650 1750 2150
-Wire Wire Line
-	1750 2150 2950 2150
-Wire Wire Line
-	2950 2150 2950 2550
-Text Label 2600 2650 0    60   ~ 0
-+5V
-Text Label 1750 1700 3    60   ~ 0
-+5V
-Wire Wire Line
-	2950 2550 2550 2550
-Wire Wire Line
-	3700 2350 3700 4850
-Wire Wire Line
-	3700 5150 3700 6350
+	3700 2350 3700 3050
+Wire Wire Line
+	3700 3050 3700 4400
+Wire Wire Line
+	3700 4400 3700 4850
+Wire Wire Line
+	3700 5150 3700 6200
+Wire Wire Line
+	3700 6200 3700 6350
+Wire Wire Line
+	3300 2350 3700 2350
 Wire Wire Line
 	3700 2350 6450 2350
-Wire Wire Line
-	6450 1950 6450 2650
-Wire Wire Line
-	6450 2650 6000 2650
 Wire Wire Line
 	5500 2950 3900 2950
 Text Label 5450 2950 2    60   ~ 0
 GND
-Text Label 6050 2650 0    60   ~ 0
-+5V
 NoConn ~ 6000 3150
 NoConn ~ 2550 3150
@@
 	4100 6700 4100 6600
 Wire Wire Line
-	3900 6600 4425 6600
+	3900 6600 4100 6600
+Wire Wire Line
+	4100 6600 4425 6600
 Wire Wire Line
 	4425 6600 4425 6750
@@
 L CP C4
 U 1 1 5E451945
-P 8150 3050
-F 0 "C4" V 8300 3050 50  0000 L CNN
-F 1 "4.7u" V 7950 3000 50  0000 L CNN
-F 2 "" H 8188 2900 50  0000 C CNN
-F 3 "" H 8150 3050 50  0000 C CNN
-	1    8150 3050
+P 8050 3050
+F 0 "C4" V 8200 3050 50  0000 L CNN
+F 1 "4.7u" V 7850 3000 50  0000 L CNN
+F 2 "" H 8088 2900 50  0000 C CNN
+F 3 "" H 8050 3050 50  0000 C CNN
+	1    8050 3050
 	0    -1   -1   0
 $EndComp
@@
 $EndComp
 Wire Wire Line
-	8300 3050 8700 3050
+	8200 3050 8400 3050
+Wire Wire Line
+	8400 3050 8600 3050
+Wire Wire Line
+	8600 3050 8700 3050
 Wire Wire Line
 	9000 3050 9400 3050
@@
 GPIO17
 Wire Wire Line
-	7850 3050 8000 3050
+	7850 3050 7900 3050
+Wire Wire Line
+	7900 3050 7900 3050
 Wire Wire Line
 	7900 2750 7900 3050
 Connection ~ 7900 3050
 Wire Wire Line
-	7550 3250 7550 4550
-Wire Wire Line
-	7550 3550 8600 3550
+	7550 3250 7550 3550
+Wire Wire Line
+	7550 3550 7550 4550
+Wire Wire Line
+	7550 3550 8400 3550
+Wire Wire Line
+	8400 3550 8600 3550
 Wire Wire Line
 	8600 3550 8600 3450
@@
 	7550 2250 7900 2250
 Wire Wire Line
-	7900 1950 7900 2450
+	7900 1950 7900 2250
+Wire Wire Line
+	7900 2250 7900 2450
 Wire Wire Line
 	6450 1950 7900 1950
+Wire Wire Line
+	7900 1950 8200 1950
 Connection ~ 7900 2250
 Connection ~ 6450 2350
@@
 	8400 4925 8400 4850
 Wire Wire Line
-	8400 4850 10500 4850
+	8400 4850 9300 4850
+Wire Wire Line
+	9300 4850 10500 4850
 Wire Wire Line
 	9300 4850 9300 5300
@@
 Text Label 7550 3650 3    60   ~ 0
 GND
+Wire Wire Line
+	3200 3050 3700 3050
+Connection ~ 3700 3050
+NoConn ~ 2550 2650
+NoConn ~ 2550 2550
+Connection ~ 3700 2350
+Wire Wire Line
+	6450 1950 6450 2350
+Wire Wire Line
+	6450 2350 6450 2550
+NoConn ~ 6000 2650
+NoConn ~ 9900 2650
+NoConn ~ 9900 2550
+Wire Wire Line
+	8200 1900 8200 1950
+Wire Wire Line
+	8200 1950 8200 4925
+Text Label 8200 2200 1    60   ~ 0
++5V
+Connection ~ 8200 1950
+Connection ~ 7900 1950
 $EndSCHEMATC

Commit message: 200426
Connections:
- net +5V: now also C2.1, JP1.4 (P4); no longer C2.2
- net GNDPWR: now also C2.2; no longer C2.1, JP1.25 (P25), JP1.9 (P9), JP2.6 (P6), JP2.9 (P9), JP4.14 (P14), JP4.6 (P6)
- no-connect marks 85 -> 91
Other:
- moved on the sheet: C1, C2, D1, L1
Changed lines of the file:
@@
 L D D1
 U 1 1 5D8B1D7E
-P 3500 5950
-F 0 "D1" V 3450 6100 50  0000 C CNN
-F 1 "1N5408" V 3850 5950 50  0000 C CNN
-F 2 "" H 3500 5950 50  0000 C CNN
-F 3 "" H 3500 5950 50  0000 C CNN
-	1    3500 5950
-	0    -1   -1   0
+P 3900 6175
+F 0 "D1" H 3900 6025 50  0000 C CNN
+F 1 "1N5408" H 3900 6325 50  0000 C CNN
+F 2 "" H 3900 6175 50  0000 C CNN
+F 3 "" H 3900 6175 50  0000 C CNN
+	1    3900 6175
+	1    0    0    -1
 $EndComp
 $Comp
@@
 	1    0    0    -1
 $EndComp
-Text Label 5450 3750 2    60   ~ 0
-GND
 Text Label 5450 3650 2    60   ~ 0
 SCLK
@@
 Text Label 8200 4925 1    60   ~ 0
 +5V
-Text Label 9950 2750 0    60   ~ 0
-GND
-Text Label 9950 3150 0    60   ~ 0
-GND
-Text Label 9150 2200 0    60   ~ 0
-GND
-Text Label 9100 4650 0    60   ~ 0
-GND
 Text Label 9350 2650 2    60   ~ 0
 GPIO02
@@
 	5200 5650 5200 6300
 Wire Wire Line
-	6000 2750 7300 2750
-Wire Wire Line
 	7300 2750 7300 5850
 Wire Wire Line
@@
 	4800 3650 5500 3650
 Wire Wire Line
-	5500 3750 4700 3750
-Wire Wire Line
-	4700 3750 4700 2250
-Wire Wire Line
-	4700 2250 3400 2250
-Wire Wire Line
 	3400 2250 3400 1275
 Wire Wire Line
@@
 	8900 4250 9400 4250
 Wire Wire Line
-	9900 2750 10200 2750
-Wire Wire Line
-	10200 2750 10200 4650
-Wire Wire Line
-	10200 4650 9100 4650
-Wire Wire Line
 	9100 4650 9100 4925
 Wire Wire Line
@@
 Wire Wire Line
 	8800 2850 9400 2850
-Wire Wire Line
-	9900 3150 10400 3150
-Wire Wire Line
-	10400 3150 10400 2200
-Wire Wire Line
-	10400 2200 9100 2200
-Wire Wire Line
-	9100 2200 9100 1900
 Wire Wire Line
 	6300 5750 6300 6300
@@
 	2150 5250 2150 6300
 Wire Wire Line
-	2050 2950 1100 2950
-Wire Wire Line
-	1100 2950 1100 5650
-Wire Wire Line
-	1100 5650 2750 5650
-Wire Wire Line
-	2750 5650 2750 6300
+	2750 3600 2750 6300
 Wire Wire Line
 	2650 6300 2650 5450
@@
 	1650 1650 1650 2250
 Wire Wire Line
-	1650 2250 2850 2250
-Wire Wire Line
-	2850 2250 2850 2750
-Wire Wire Line
-	2850 2750 2550 2750
+	1650 2250 6975 2250
 Text Notes 1900 950  0    60   ~ 0
 Console
@@
 NoConn ~ 2050 2750
 NoConn ~ 2050 2850
-Text Label 2000 2950 2    60   ~ 0
-GND
 NoConn ~ 2050 3050
 Text Label 2000 3150 2    60   ~ 0
@@
 Text Label 2600 2850 0    60   ~ 0
 TXD
-Text Label 2600 2750 0    60   ~ 0
-GND
 Text Label 2050 6250 1    60   ~ 0
 +5V
@@
 Text Notes 5650 6800 0    60   ~ 0
 LEDs
-Text Notes 8500 5700 0    60   ~ 0
+Text Notes 8450 5700 0    60   ~ 0
 Outputs
-Text Notes 8450 1400 0    60   ~ 0
+Text Notes 8450 1225 0    60   ~ 0
 Outputs
 Text Notes 5300 950  0    60   ~ 0
@@
 	3700 6700 3700 6650
 Wire Wire Line
-	3900 2950 3900 3850
-Wire Wire Line
-	3900 3850 3900 4550
-Wire Wire Line
-	3900 4550 3900 5650
-Wire Wire Line
-	3900 5650 3900 6600
+	4100 2250 4100 6700
 Wire Wire Line
 	3900 6600 3900 6700
-Wire Wire Line
-	3500 6100 3500 6200
-Wire Wire Line
-	3500 6200 3700 6200
-Wire Wire Line
-	3450 4400 3700 4400
-Wire Wire Line
-	3700 4400 4150 4400
-Connection ~ 3700 6200
-Wire Wire Line
-	3500 5800 3500 5650
-Wire Wire Line
-	3500 5650 3900 5650
-Wire Wire Line
-	3450 3850 3900 3850
-Wire Wire Line
-	3900 3850 4150 3850
-Connection ~ 3900 5650
 Text Notes 3575 7275 0    60   ~ 0
   Power in\n(5V 2.5A DC)
 Wire Wire Line
-	3700 2350 3700 3050
-Wire Wire Line
-	3700 3050 3700 4400
-Wire Wire Line
-	3700 4400 3700 4850
-Wire Wire Line
-	3700 5150 3700 6200
-Wire Wire Line
-	3700 6200 3700 6350
-Wire Wire Line
-	3300 2350 3700 2350
-Wire Wire Line
-	3700 2350 6450 2350
-Wire Wire Line
-	5500 2950 3900 2950
-Text Label 5450 2950 2    60   ~ 0
-GND
+	3700 2350 3700 5050
+Wire Wire Line
+	3700 5350 3700 6350
+Wire Wire Line
+	3300 2350 6450 2350
 NoConn ~ 6000 3150
 NoConn ~ 2550 3150
@@
 $EndComp
 Wire Wire Line
-	4100 6700 4100 6600
-Wire Wire Line
-	3900 6600 4100 6600
-Wire Wire Line
-	4100 6600 4425 6600
+	3900 6600 4425 6600
 Wire Wire Line
 	4425 6600 4425 6750
@@
 $EndComp
 Wire Wire Line
-	8200 3050 8400 3050
-Wire Wire Line
-	8400 3050 8600 3050
-Wire Wire Line
-	8600 3050 8700 3050
+	8200 3050 8700 3050
 Wire Wire Line
 	9000 3050 9400 3050
@@
 	7850 3050 7900 3050
 Wire Wire Line
-	7900 3050 7900 3050
-Wire Wire Line
-	7900 2750 7900 3050
+	7900 3050 7900 2750
 Connection ~ 7900 3050
 Wire Wire Line
-	7550 3250 7550 3550
-Wire Wire Line
-	7550 3550 7550 4550
-Wire Wire Line
-	7550 3550 8400 3550
-Wire Wire Line
-	8400 3550 8600 3550
+	7300 3550 8600 3550
 Wire Wire Line
 	8600 3550 8600 3450
@@
 	7550 2250 7900 2250
 Wire Wire Line
-	7900 1950 7900 2250
-Wire Wire Line
-	7900 2250 7900 2450
-Wire Wire Line
-	6450 1950 7900 1950
-Wire Wire Line
-	7900 1950 8200 1950
+	7900 1950 7900 2450
+Wire Wire Line
+	6450 1950 8200 1950
 Connection ~ 7900 2250
 Connection ~ 6450 2350
-Wire Wire Line
-	7550 4550 3900 4550
-Connection ~ 3900 4550
 Connection ~ 7550 3550
 $Comp
 L CP C1
 U 1 1 5E453D9A
-P 3450 4150
-F 0 "C1" H 3550 4050 50  0000 L CNN
-F 1 "1000u" H 3350 4500 50  0000 L CNN
-F 2 "" H 3488 4000 50  0000 C CNN
-F 3 "" H 3450 4150 50  0000 C CNN
-	1    3450 4150
-	-1   0    0    1
+P 3900 4825
+F 0 "C1" V 3900 5125 50  0000 L CNN
+F 1 "1000u" V 3700 4725 50  0000 L CNN
+F 2 "" H 3938 4675 50  0000 C CNN
+F 3 "" H 3900 4825 50  0000 C CNN
+	1    3900 4825
+	0    -1   -1   0
 $EndComp
 $Comp
 L C C2
 U 1 1 5E45409D
-P 4150 4150
-F 0 "C2" H 3990 4260 50  0000 L CNN
-F 1 "100n" H 4060 3810 50  0000 L CNN
-F 2 "" H 4188 4000 50  0000 C CNN
-F 3 "" H 4150 4150 50  0000 C CNN
-	1    4150 4150
-	1    0    0    -1
-$EndComp
-Wire Wire Line
-	4150 3850 4150 4000
-Wire Wire Line
-	4150 4400 4150 4300
+P 3900 4525
+F 0 "C2" V 3900 4825 50  0000 L CNN
+F 1 "100n" V 4075 4425 50  0000 L CNN
+F 2 "" H 3938 4375 50  0000 C CNN
+F 3 "" H 3900 4525 50  0000 C CNN
+	1    3900 4525
+	0    -1   -1   0
+$EndComp
 $Comp
 L L_Core_Ferrite L1
 U 1 1 5E4582AE
-P 3700 5000
-F 0 "L1" H 3850 5000 50  0000 C CNN
-F 1 "L_Core_Ferrite" V 3810 5000 50  0001 C CNN
-F 2 "" H 3700 5000 50  0000 C CNN
-F 3 "" H 3700 5000 50  0000 C CNN
-	1    3700 5000
+P 3700 5200
+F 0 "L1" H 3850 5200 50  0000 C CNN
+F 1 "L_Core_Ferrite" V 3810 5200 50  0001 C CNN
+F 2 "" H 3700 5200 50  0000 C CNN
+F 3 "" H 3700 5200 50  0000 C CNN
+	1    3700 5200
 	-1   0    0    1
 $EndComp
-Wire Wire Line
-	3450 3850 3450 4000
-Wire Wire Line
-	3450 4400 3450 4300
-Connection ~ 3700 4400
-Connection ~ 3900 3850
 $Comp
 L SWITCH_1P SW1
@@
 	8400 4925 8400 4850
 Wire Wire Line
-	8400 4850 9300 4850
-Wire Wire Line
-	9300 4850 10500 4850
+	8400 4850 10500 4850
 Wire Wire Line
 	9300 4850 9300 5300
@@
 Text Label 10450 5300 2    60   ~ 0
 +5V
-Text Label 7900 2200 1    60   ~ 0
-+5V
 NoConn ~ 2450 1650
 NoConn ~ 2350 1650
@@
 NoConn ~ 1950 1650
 NoConn ~ 1850 1650
-Connection ~ 3900 6600
 Connection ~ 4100 6600
 Wire Wire Line
@@
 Text Label 9325 2000 2    60   ~ 0
 +5V
-Text Label 7550 3650 3    60   ~ 0
-GND
 Wire Wire Line
 	3200 3050 3700 3050
@@
 Connection ~ 3700 2350
 Wire Wire Line
-	6450 1950 6450 2350
-Wire Wire Line
-	6450 2350 6450 2550
-NoConn ~ 6000 2650
+	6450 1950 6450 2650
 NoConn ~ 9900 2650
 NoConn ~ 9900 2550
 Wire Wire Line
-	8200 1900 8200 1950
-Wire Wire Line
-	8200 1950 8200 4925
-Text Label 8200 2200 1    60   ~ 0
-+5V
+	8200 1900 8200 4925
 Connection ~ 8200 1950
 Connection ~ 7900 1950
+Wire Wire Line
+	2750 3600 4100 3600
+Connection ~ 4100 3600
+Connection ~ 3400 2250
+Wire Wire Line
+	6450 2650 6000 2650
+Connection ~ 6450 2550
+Wire Wire Line
+	6000 2750 6525 2750
+Wire Wire Line
+	6525 2750 6525 2250
+Text Label 6050 2650 0    60   ~ 0
++5V
+Wire Wire Line
+	6975 2250 6975 2750
+Wire Wire Line
+	6975 2750 7300 2750
+Connection ~ 6525 2250
+Wire Wire Line
+	7550 3250 7550 3550
+Connection ~ 7300 3550
+Wire Wire Line
+	7300 4650 10400 4650
+Connection ~ 7300 4650
+Wire Wire Line
+	10400 4650 10400 2200
+Wire Wire Line
+	10400 2200 9100 2200
+Wire Wire Line
+	9100 2200 9100 1900
+Connection ~ 9100 4650
+NoConn ~ 9900 2750
+NoConn ~ 9900 3150
+NoConn ~ 5500 2950
+NoConn ~ 5500 3750
+NoConn ~ 2550 2750
+NoConn ~ 2050 2950
+NoConn ~ 1750 1650
+Wire Wire Line
+	3750 4525 3700 4525
+Connection ~ 3700 4525
+Wire Wire Line
+	3750 4825 3700 4825
+Connection ~ 3700 4825
+Wire Wire Line
+	4050 4825 4100 4825
+Connection ~ 4100 4825
+Wire Wire Line
+	4050 4525 4100 4525
+Connection ~ 4100 4525
+Wire Wire Line
+	3750 6175 3700 6175
+Connection ~ 3700 6175
+Wire Wire Line
+	4050 6175 4100 6175
+Connection ~ 4100 6175
+Connection ~ 4100 2250
 $EndSCHEMATC
