File: cad_files/mm5d-sch/u4.sch (KiCad schematic (older format))
At the start: 30 parts, among them SW401 SWITCH_1P

Commit message: 200426
Parts:
- R401, R406, R407, R408, R409, R410, R411, R412, R413, R414: value 220 -> 330
Changed lines of the file:
@@
 P 6300 2850
 F 0 "R406" V 6200 2800 50  0000 C CNN
-F 1 "220" V 6400 2900 50  0000 C CNN
+F 1 "330" V 6400 2900 50  0000 C CNN
 F 2 "" V 6230 2850 50  0000 C CNN
 F 3 "" H 6300 2850 50  0000 C CNN
@@
 P 6600 2850
 F 0 "R407" V 6500 2800 50  0000 C CNN
-F 1 "220" V 6700 2900 50  0000 C CNN
+F 1 "330" V 6700 2900 50  0000 C CNN
 F 2 "" V 6530 2850 50  0000 C CNN
 F 3 "" H 6600 2850 50  0000 C CNN
@@
 P 6900 2850
 F 0 "R408" V 6800 2800 50  0000 C CNN
-F 1 "220" V 7000 2900 50  0000 C CNN
+F 1 "330" V 7000 2900 50  0000 C CNN
 F 2 "" V 6830 2850 50  0000 C CNN
 F 3 "" H 6900 2850 50  0000 C CNN
@@
 P 7200 2850
 F 0 "R409" V 7100 2800 50  0000 C CNN
-F 1 "220" V 7300 2900 50  0000 C CNN
+F 1 "330" V 7300 2900 50  0000 C CNN
 F 2 "" V 7130 2850 50  0000 C CNN
 F 3 "" H 7200 2850 50  0000 C CNN
@@
 P 7700 2850
 F 0 "R410" V 7600 2800 50  0000 C CNN
-F 1 "220" V 7800 2900 50  0000 C CNN
+F 1 "330" V 7800 2900 50  0000 C CNN
 F 2 "" V 7630 2850 50  0000 C CNN
 F 3 "" H 7700 2850 50  0000 C CNN
@@
 P 8000 2850
 F 0 "R411" V 7900 2800 50  0000 C CNN
-F 1 "220" V 8100 2900 50  0000 C CNN
+F 1 "330" V 8100 2900 50  0000 C CNN
 F 2 "" V 7930 2850 50  0000 C CNN
 F 3 "" H 8000 2850 50  0000 C CNN
@@
 P 8300 2850
 F 0 "R412" V 8200 2800 50  0000 C CNN
-F 1 "220" V 8400 2900 50  0000 C CNN
+F 1 "330" V 8400 2900 50  0000 C CNN
 F 2 "" V 8230 2850 50  0000 C CNN
 F 3 "" H 8300 2850 50  0000 C CNN
@@
 P 8600 2850
 F 0 "R413" V 8500 2800 50  0000 C CNN
-F 1 "220" V 8700 2900 50  0000 C CNN
+F 1 "330" V 8700 2900 50  0000 C CNN
 F 2 "" V 8530 2850 50  0000 C CNN
 F 3 "" H 8600 2850 50  0000 C CNN
@@
 P 9100 2850
 F 0 "R414" V 9000 2800 50  0000 C CNN
-F 1 "220" V 9200 2900 50  0000 C CNN
+F 1 "330" V 9200 2900 50  0000 C CNN
 F 2 "" V 9030 2850 50  0000 C CNN
 F 3 "" H 9100 2850 50  0000 C CNN
@@
 P 4500 2850
 F 0 "R401" V 4400 2800 50  0000 C CNN
-F 1 "220" V 4600 2900 50  0000 C CNN
+F 1 "330" V 4600 2900 50  0000 C CNN
 F 2 "" V 4430 2850 50  0000 C CNN
 F 3 "" H 4500 2850 50  0000 C CNN
