File: cad_files/connecting/connecting.sch (KiCad schematic (older format))
At the start: 60 parts, among them P1 SCREW_CONN_1, P10 SCREW_CONN_1, P11 SCREW_CONN_1, P12 SCREW_CONN_1, P13 SCREW_CONN_1, P14 SCREW_CONN_1, P15 SCREW_CONN_1, P16 SCREW_CONN_1, P17 SCREW_CONN_1, P18 SCREW_CONN_1, P19 SCREW_CONN_1, P2 SCREW_CONN_1, P20 SCREW_CONN_1, P21 SCREW_CONN_1, P22 SCREW_CONN_1, P23 SCREW_CONN_1, P24 SCREW_CONN_1, P25 SCREW_CONN_1, P26 SCREW_CONN_1, P27 SCREW_CONN_1, P29 SCREW_CONN_1, P3 SCREW_CONN_1, P30 SCREW_CONN_1, P32 SCREW_CONN_1, P33 SCREW_CONN_1, P4 SCREW_CONN_1, P5 SCREW_CONN_1, P6 SCREW_CONN_1, P7 SCREW_CONN_1, P8 SCREW_CONN_1, P9 SCREW_CONN_1, SW1 SWITCH_2P, SW2 SWITCH_2P, SW3 SWITCH_1P_CLOSED, SW4 SWITCH_1P_CLOSED, U1 DHT11, U2 DHT11

Commit message: 200218
Other:
- note added: "Signal lamps"
- note removed: "Signalling\n lamp"
Changed lines of the file:
@@
 Sheet 1 1
 Title "MM4A Electrical distribution and switching unit"
-Date "2019-09-19"
-Rev "190919"
+Date "2019-11-01"
+Rev "191101"
 Comp "Pozsar Zsolt -  http://www.szerafingomba.hu"
 Comment1 "Connecting of unit"
 Comment2 ""
 Comment3 ""
-Comment4 "Draw no.: 59/5/6"
+Comment4 "Draw no.: 59/5/5"
 $EndDescr
 $Comp
@@
 Text Notes 7450 4500 0    60   ~ 0
 Solenoid\nof valve
-Text Notes 8325 4500 0    60   ~ 0
-Signalling\n  lamp
+Text Notes 9050 3800 0    60   ~ 0
+Signal lamps
 Text Notes 9075 4650 0    60   ~ 0
 G     Y     R

Commit message: 200219
Parts:
- removed P9: SCREW_CONN_1, ~, symbol SCREW_CONN_1
- removed R1, R2: 4.7k, symbol R
- removed U1: DHT11, symbol DHT11
- U1: renamed from U2; value DHT11 -> DHT22
- renumbered P1 to J1/1, P2 to J1/2, P3 to J1/3, P5 to U5/J501/1, P6 to U5/J501/2, P7 to U5/J501/3, P8 to U5/J501/4, P4 to U5/J501/5, P11 to U5/J502/1, P10 to U5/J502/2, P12 to U5/J502/3, P14 to U6/K1/C, P15 to U6/K1/NO, P17 to U6/K2/C, P18 to U6/K2/NO, P20 to U6/K3/C, P21 to U6/K3/NO, P23 to U6/K4/C, P24 to U6/K4/NO, P26 to U7/K1/C, P27 to U7/K1/NO, P29 to U7/K2/C, P30 to U7/K2/NO, P32 to U7/K3/C, P33 to U7/K3/NO
Other:
- note added: "+"
- note added: "-"
- note added: "Data"
- note added: "In1"
- note added: "In2"
- note added: "In3"
- note added: "In4"
- note added: "Manual on/off"
- note added: "Out1"
- note added: "Out2"
- note added: "Out3"
- note added: "Out4"
- note added: "Out5"
- note added: "Out6"
- note added: "Out7"
- note added: "T/RH sensor"
- note removed: "IN1"
- note removed: "IN2"
- note removed: "IN3"
- note removed: "IN4"
- note removed: "OUT1"
- note removed: "OUT2"
- note removed: "OUT3"
- note removed: "OUT4"
- note removed: "OUT5"
- note removed: "OUT6"
- note removed: "OUT7"
- note removed: "Sensors"
- moved on the sheet: U1, U5/J502/1

Commit message: 230323
Parts:
- added U7/K2/NC, U7/K3/NC: SCREW_CONN_1, ~, symbol SCREW_CONN_1
- renumbered U7/K1/NO to U7/K1/NC
Connections:
- net 24V_L: no longer U7/K1/C.1, U7/K3/C.1
- net at La1.2 (+): now also U7/K3/NC.1; no longer U7/K1/NC.1
- net at U5/J502/1.1: now also U7/K1/C.1; no longer U1.1 (VCC)
- new net: U1.1 (VCC), U7/K1/NC.1
- new net: U7/K2/NC.1, U7/K3/C.1
Changed lines of the file:
@@
 	1250 825  1250 1725
 Wire Wire Line
-	8475 1625 8475 2050
-Wire Wire Line
-	8475 2050 8475 2500
+	8475 1625 8475 2500
 Wire Wire Line
 	8225 1625 8225 2500
@@
 	7975 1625 7975 3425
 Wire Wire Line
-	7975 3425 8225 3425
-Wire Wire Line
-	8225 3425 8475 3425
+	7975 3425 8475 3425
 Wire Wire Line
 	8475 3425 8475 3350
@@
 Connection ~ 8225 3425
 Wire Wire Line
-	9375 1625 9375 2150
-Wire Wire Line
-	9375 2150 9375 2500
+	9375 1625 9375 2500
 Wire Wire Line
 	9125 1625 9125 2500
@@
 	8875 1625 8875 3425
 Wire Wire Line
-	8875 3425 9125 3425
-Wire Wire Line
-	9125 3425 9375 3425
+	8875 3425 9375 3425
 Wire Wire Line
 	9375 3425 9375 3350
@@
 	6450 5000 5800 5000
 Wire Wire Line
-	5800 5000 5800 5200
-Wire Wire Line
-	5800 5200 5800 5475
+	5800 5000 5800 5475
 Wire Wire Line
 	7100 5200 7100 5475
 Wire Wire Line
-	5800 5200 6450 5200
-Wire Wire Line
-	6450 5200 7100 5200
+	5800 5200 7100 5200
 Connection ~ 5800 5200
 Wire Wire Line
@@
 $EndComp
 $Comp
-L SCREW_CONN_1 U7/K1/NO
+L SCREW_CONN_1 U7/K1/NC
 U 1 1 5D87D8F6
 P 8650 5625
-F 0 "U7/K1/NO" H 8730 5625 40  0000 L CNN
+F 0 "U7/K1/NC" H 8730 5625 40  0000 L CNN
 F 1 "SCREW_CONN_1" H 8650 5680 30  0001 C CNN
 F 2 "~" H 8650 5625 60  0000 C CNN
@@
 	7750 5475 7750 5200
 Wire Wire Line
-	7750 5200 8400 5200
-Wire Wire Line
-	8400 5200 9050 5200
-Wire Wire Line
-	9050 5200 9700 5200
-Wire Wire Line
-	9700 5200 10450 5200
-Wire Wire Line
-	8400 5200 8400 5475
+	7750 5200 10450 5200
 Wire Wire Line
 	9050 5200 9050 5475
-Connection ~ 8400 5200
-Wire Wire Line
-	9700 5200 9700 5475
 Connection ~ 9050 5200
 Wire Notes Line
@@
 	9025 4225 9025 4150
 Wire Wire Line
-	9025 4150 9300 4150
-Wire Wire Line
-	9300 4150 9575 4150
+	9025 4150 9575 4150
 Wire Wire Line
 	9575 4150 9575 4225
 Wire Wire Line
-	9300 3900 9300 4150
-Wire Wire Line
-	9300 4150 9300 4225
+	9300 3900 9300 4225
 Connection ~ 9300 4150
-Wire Wire Line
-	8650 5475 8650 5100
-Wire Wire Line
-	8650 5100 9025 5100
-Wire Wire Line
-	9025 5100 9025 4625
 Wire Wire Line
 	9950 5475 9950 5100
@@
 	8000 5475 8000 4575
 Wire Wire Line
-	8000 3900 9300 3900
-Wire Wire Line
-	9300 3900 10075 3900
+	8000 3900 10075 3900
 Wire Wire Line
 	8000 3900 8000 4275
@@
 Text Notes 10225 4675 0    60   ~ 0
     Mains\n24 V 50/60 Hz\n    PELV
-Connection ~ 9700 5200
 Wire Wire Line
 	10075 4850 10450 4850
@@
 G     Y     R
 Wire Wire Line
-	3250 1625 3250 3925
-Wire Wire Line
-	3250 3925 3250 5475
+	3250 1625 3250 5475
 Wire Wire Line
 	3500 5475 3500 1625
@@
 	4000 4225 4000 3925
 Wire Wire Line
-	3250 3925 4000 3925
-Wire Wire Line
-	4000 3925 4250 3925
+	3250 3925 4250 3925
 Connection ~ 3250 3925
 Wire Wire Line
@@
 Wire Wire Line
 	5400 2625 4650 2625
-Wire Wire Line
-	4650 2625 4650 5475
 Text Notes 4850 6200 0    60   ~ 0
 Data
@@
 Text Notes 4975 2500 0    60   ~ 0
 T/RH sensor
+$Comp
+L SCREW_CONN_1 U7/K2/NC
+U 1 1 641C7442
+P 9175 5625
+F 0 "U7/K2/NC" H 9255 5625 40  0000 L CNN
+F 1 "SCREW_CONN_1" H 9175 5680 30  0001 C CNN
+F 2 "~" H 9175 5625 60  0000 C CNN
+F 3 "~" H 9175 5625 60  0000 C CNN
+	1    9175 5625
+	0    -1   1    0
+$EndComp
+$Comp
+L SCREW_CONN_1 U7/K3/NC
+U 1 1 641C7520
+P 9825 5625
+F 0 "U7/K3/NC" H 9905 5625 40  0000 L CNN
+F 1 "SCREW_CONN_1" H 9825 5680 30  0001 C CNN
+F 2 "~" H 9825 5625 60  0000 C CNN
+F 3 "~" H 9825 5625 60  0000 C CNN
+	1    9825 5625
+	0    -1   1    0
+$EndComp
+Wire Wire Line
+	9175 5475 9175 5275
+Wire Wire Line
+	9175 5275 9700 5275
+Wire Wire Line
+	9700 5275 9700 5475
+Wire Wire Line
+	9825 5475 9825 5025
+Wire Wire Line
+	9825 5025 9025 5025
+Wire Wire Line
+	9025 5025 9025 4625
+Wire Wire Line
+	8400 5475 8400 4875
+Wire Wire Line
+	8400 4875 4650 4875
+Wire Wire Line
+	4650 4875 4650 5475
+Wire Wire Line
+	4650 2625 4650 4750
+Wire Wire Line
+	4650 4750 8650 4750
+Wire Wire Line
+	8650 4750 8650 5475
 $EndSCHEMATC
